Commit message: ready for test

File: nj_220_2_7_gazebo/urdf/nj_220_2_7.xacro (robot description, xacro)
@@ -163,238 +163,4 @@
       effort="${joint_2_eff_limit}"
       velocity="${joint_2_vel_limit}" />
-  </joint>
-  <link name="${prefix}link_3">
-    <inertial>
-      <origin
-        xyz="-0.04239 0.01939 0.2104"
-        rpy="0 0 0" />
-      <mass
-        value="303.81" />
-      <inertia
-        ixx="24.45402173"
-        ixy="-0.58037596"
-        ixz="-2.46563321"
-        iyy="20.71802091"
-        iyz="2.40454026"
-        izz="9.01610712" />
-    </inertial>
-    <visual>
-      <origin
-        xyz="0 0 0"
-        rpy="0 0 0" />
-      <geometry>
-        <mesh
-          filename="package://nj_220_2_7_gazebo/meshes/link_3.STL" />
-      </geometry>
-      <material
-        name="">
-        <color
-          rgba="1 0 0 1" />
-      </material>
-    </visual>
-    <collision>
-      <origin
-        xyz="0 0 0"
-        rpy="0 0 0" />
-      <geometry>
-        <mesh
-          filename="package://nj_220_2_7_gazebo/meshes/link_3.STL" />
-      </geometry>
-    </collision>
-  </link>
-  <joint name="${prefix}joint_3" type="revolute">
-    <origin
-      xyz="0 0 0"
-      rpy="0 0 0" />
-    <parent
-      link="${prefix}link_3_virtual" />
-    <child
-      link="${prefix}link_3" />
-    <axis
-      xyz="0 -1 0" />
-    <limit
-      lower="-4.468042885"
-      upper="0.174532925"
-      effort="${joint_3_eff_limit}"
-      velocity="${joint_3_vel_limit}" />
-  </joint>
-  <link name="${prefix}link_4">
-    <inertial>
-      <origin
-        xyz="0.71228 -0.02567 -0.00003"
-        rpy="0 0 0" />
-      <mass
-        value="90.963" />
-      <inertia
-        ixx="0.68929228290"
-        ixy="-2.39235486446"
-        ixz="-0.00192589885"
-        iyy="58.11987131958"
-        iyz="-0.00017654018"
-        izz="58.29818388998" />
-    </inertial>
-    <visual>
-      <origin
-        xyz="0 0 0"
-        rpy="0 0 0" />
-      <geometry>
-        <mesh
-          filename="package://nj_220_2_7_gazebo/meshes/link_4.STL" />
-      </geometry>
-      <material
-        name="">
-        <color
-          rgba="1 0 0 1" />
-      </material>
-    </visual>
-    <collision>
-      <origin
-        xyz="0 0 0"
-        rpy="0 0 0" />
-      <geometry>
-        <mesh
-          filename="package://nj_220_2_7_gazebo/meshes/link_4.STL" />
-      </geometry>
-    </collision>
-  </link>
-  <joint name="${prefix}joint_4" type="revolute">
-    <origin
-      xyz="0.105 0 0.25"
-      rpy="0 0 0" />
-    <parent
-      link="${prefix}link_3" />
-    <child
-      link="${prefix}link_4" />
-    <axis
-      xyz="1 0 0" />
-    <limit
-      lower="-6.2831853"
-      upper="6.2831853"
-      effort="${joint_4_eff_limit}"
-      velocity="${joint_4_vel_limit}" />
-  </joint>
-  <link name="${prefix}link_5">
-    <inertial>
-      <origin
-        xyz="0.09375 0.01506 0.00002"
-        rpy="0 0 0" />
-      <mass
-        value="50.615" />
-      <inertia
-        ixx="0.67974396"
-        ixy="0.04508972"
-        ixz="0.00009980"
-        iyy="0.83229961"
-        iyz="0.00011851"
-        izz="1.32231171" />
-    </inertial>
-    <visual>
-      <origin
-        xyz="0 0 0"
-        rpy="0 0 0" />
-      <geometry>
-        <mesh
-          filename="package://nj_220_2_7_gazebo/meshes/link_5.STL" />
-      </geometry>
-      <material
-        name="">
-        <color
-          rgba="1 0 0 1" />
-      </material>
-    </visual>
-    <collision>
-      <origin
-        xyz="0 0 0"
-        rpy="0 0 0" />
-      <geometry>
-        <mesh
-          filename="package://nj_220_2_7_gazebo/meshes/link_5.STL" />
-      </geometry>
-    </collision>
-  </link>
-  <joint name="${prefix}joint_5" type="revolute">
-    <origin
-      xyz="1.02033 0 0"
-      rpy="0 0 0" />
-    <parent
-      link="${prefix}link_4" />
-    <child
-      link="${prefix}link_5" />
-    <axis
-      xyz="0 1 0" />
-    <limit
-      lower="-2.1816"
-      upper="2.1816"
-      effort="${joint_5_eff_limit}"
-      velocity="${joint_5_vel_limit}" />
-  </joint>
-  <link name="${prefix}link_6">
-    <inertial>
-      <origin
-        xyz="0.0058594 -0.00060952 -5.99E-05"
-        rpy="0 0 0" />
-      <mass
-        value="5.3437" />
-      <inertia
-        ixx="0.02913604"
-        ixy="-0.00000822"
-        ixz="-0.00000086"
-        iyy="0.01533002"
-        iyz="0.00000585"
-        izz="0.01518874" />
-    </inertial>
-    <visual>
-      <origin
-        xyz="0 0 0"
-        rpy="0 0 0" />
-      <geometry>
-        <mesh
-          filename="package://nj_220_2_7_gazebo/meshes/link_6.STL" />
-      </geometry>
-      <material
-        name="">
-        <color
-          rgba="0.25098 0.25098 0.25098 1" />
-      </material>
-    </visual>
-    <collision>
-      <origin
-        xyz="0 0 0"
-        rpy="0 0 0" />
-      <geometry>
-        <mesh
-          filename="package://nj_220_2_7_gazebo/meshes/link_6.STL" />
-      </geometry>
-    </collision>
-  </link>
-  <joint name="${prefix}joint_6" type="revolute">
-    <origin
-      xyz="0.2085 0 0"
-      rpy="0 0 0" />
-    <parent
-      link="${prefix}link_5" />
-    <child
-      link="${prefix}link_6" />
-    <axis
-      xyz="1 0 0" />
-    <limit
-      lower="-6.2831853"
-      upper="6.2831853"
-      effort="${joint_6_eff_limit}"
-      velocity="${joint_6_vel_limit}" />
-  </joint>
-  <link name="${prefix}link_3_virtual">
-   </link>
-  <joint name="${prefix}joint_2m" type="revolute">
-     <origin xyz="0 0 1.175" rpy="0 0 0" />
-     <parent link="${prefix}link_2" />
-     <child link="${prefix}link_3_virtual" />
-     <axis xyz="0 1 0" />
-     <mimic joint="${prefix}joint_2" multiplier="-1" offset="0" />
-     <limit
-       lower="-6.2831853"
-       upper="6.2831853"
-       effort="100000"
-       velocity="${joint_6_vel_limit}" />
   </joint>
   <link name="${prefix}link_2_1">
@@ -437,5 +203,5 @@
      </collision>
    </link>
-  <joint name="${prefix}joint_2_1" type="revolute">
+  <joint name="${prefix}joint_3" type="revolute">
      <origin xyz="0.400 -0.1945 0.499" rpy="1.570796327 0.087266 3.141592654" />
      <parent link="${prefix}link_1" />
@@ -443,12 +209,44 @@
      <axis xyz="0 0 1" />
      <limit
-       lower="-6.2831853"
-       upper="6.2831853"
-       effort="0"
-       velocity="0" />
-       <mimic joint="${prefix}joint_3" multiplier="-1" offset="0" />
-   </joint>
-  <link name="${prefix}link_2_2_virtual"></link>
-  <joint name="${prefix}joint_2_2" type="continuous">
+       lower="-4.468042885"
+       upper="0.174532925"
+       effort="${joint_3_eff_limit}"
+       velocity="${joint_3_vel_limit}" />
+  </joint>
+  <link name="${prefix}link_2_2">
+     <inertial>
+       <origin
+         xyz="0.06443 0.51885 0.01485"
+         rpy="0 0 0" />
+       <mass
+         value="60.72" />
+       <inertia
+         ixx="21.93937071"
+         ixy="1.89190480"
+         ixz="0.05733724"
+         iyy="0.41028863"
+         iyz="0.47064670"
+         izz="22.27041146" />
+     </inertial>
+     <visual>
+       <origin
+         xyz="0 0 0"
+         rpy="0 0 0" />
+       <geometry>
+         <mesh
+           filename="package://nj_220_2_7_gazebo/meshes/link_2_2.STL" />
+       </geometry>
+     </visual>
+     <collision>
+       <origin
+         xyz="0 0 0"
+         rpy="0 0 0" />
+       <geometry>
+         <mesh
+           filename="package://nj_220_2_7_gazebo/meshes/link_2_2.STL" />
+       </geometry>
+     </collision>
+  </link>
+  <joint name="${prefix}joint_2_1" type="continuous">
     <origin
       xyz="0.350 0 0.015"
@@ -457,51 +255,9 @@
       link="${prefix}link_2_1" />
     <child
-      link="${prefix}link_2_2_virtual" />
+      link="${prefix}link_2_2" />
     <axis
       xyz="0 0 1" />
-    <mimic joint="${prefix}joint_3" multiplier="1" offset="0"/>
-  </joint>
-  <link name="${prefix}link_2_2">
-    <inertial>
-      <origin
-        xyz="0.06443 0.51885 0.01485"
-        rpy="0 0 0" />
-      <mass
-        value="60.72" />
-      <inertia
-        ixx="21.93937071"
-        ixy="1.89190480"
-        ixz="0.05733724"
-        iyy="0.41028863"
-        iyz="0.47064670"
-        izz="22.27041146" />
-    </inertial>
-    <visual>
-      <origin
-        xyz="0 0 0"
-        rpy="0 0 0" />
-      <geometry>
-        <mesh
-          filename="package://nj_220_2_7_gazebo/meshes/link_2_2.STL" />
-      </geometry>
-    </visual>
-    <collision>
-      <origin
-        xyz="0 0 0"
-        rpy="0 0 0" />
-      <geometry>
-        <mesh
-          filename="package://nj_220_2_7_gazebo/meshes/link_2_2.STL" />
-      </geometry>
-    </collision>
-  </link>
-  <joint name="${prefix}joint_2_3" type="continuous">
-    <origin xyz="0.0 0.0 0.0" rpy="0 0 0" />
-    <parent link="${prefix}link_2_2_virtual" />
-    <child link="${prefix}link_2_2" />
-    <axis xyz="0 0 1" />
-    <mimic joint="${prefix}joint_2" multiplier="1" offset="0"/>
-  </joint>
-  <link name="${prefix}flange">
+  </joint>
+  <link name="${prefix}link_2_3">
     <inertial>
       <origin xyz="0 0 0" rpy="0 0 0" />
@@ -516,4 +272,248 @@
     </inertial>
   </link>
+  <joint name="${prefix}joint_2_2" type="continuous">
+    <origin xyz="0.0 1.175 0.0" rpy="0 0 0" />
+    <parent link="${prefix}link_2_2" />
+    <child link="${prefix}link_2_3" />
+    <axis xyz="0 0 1" />
+  </joint>
+  <link name="${prefix}link_3">
+    <inertial>
+      <origin
+        xyz="-0.04239 0.01939 0.2104"
+        rpy="0 0 0" />
+      <mass
+        value="303.81" />
+      <inertia
+        ixx="24.45402173"
+        ixy="-0.58037596"
+        ixz="-2.46563321"
+        iyy="20.71802091"
+        iyz="2.40454026"
+        izz="9.01610712" />
+    </inertial>
+    <visual>
+      <origin
+        xyz="0 0 0"
+        rpy="0 0 0" />
+      <geometry>
+        <mesh
+          filename="package://nj_220_2_7_gazebo/meshes/link_3.STL" />
+      </geometry>
+      <material
+        name="">
+        <color
+          rgba="1 0 0 1" />
+      </material>
+    </visual>
+    <collision>
+      <origin
+        xyz="0 0 0"
+        rpy="0 0 0" />
+      <geometry>
+        <mesh
+          filename="package://nj_220_2_7_gazebo/meshes/link_3.STL" />
+      </geometry>
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