Commit message: Testing phase

File: nj_220_2_7_description/urdf/nj_220_2_7.xacro (robot description, xacro)
@@ -1,6 +1,6 @@
 <?xml version="1.0" ?>
 <robot xmlns:xacro="http://ros.org/wiki/xacro">
-<!-- <xacro:macro name="nj_220_2_7" params="prefix:='' interface:=hardware_interface/EffortJointInterface"> -->
-<xacro:macro name="nj_220_2_7" params="prefix:='' interface:=hardware_interface/PositionJointInterface">
+<xacro:macro name="nj_220_2_7" params="prefix:='' interface:=hardware_interface/EffortJointInterface">
+<!-- <xacro:macro name="nj_220_2_7" params="prefix:='' interface:=hardware_interface/PositionJointInterface"> -->
   <xacro:property name="joint_1_vel_limit" value="1.74533" />    <!--  100°/s -->
   <xacro:property name="joint_2_vel_limit" value="1.5708"  />    <!--  90°/s -->
@@ -384,6 +384,5 @@
       velocity="${joint_6_vel_limit}" />
   </joint>
-  <!-- Parallel Linkages  -->
-   <link name="${prefix}link_3_virtual">
+  <link name="${prefix}link_3_virtual">
      <inertial>
        <origin xyz="0 0 0" rpy="0 0 0" />
@@ -398,5 +397,5 @@
      </inertial>
    </link>
-   <joint name="${prefix}joint_2m" type="continuous">
+  <joint name="${prefix}joint_2m" type="revolute">
      <origin xyz="0 1.175 0.0955" rpy="3.1416 0 -1.5708" />
      <parent link="${prefix}link_2" />
@@ -404,6 +403,152 @@
      <axis xyz="0 0 -1" />
      <mimic joint="${prefix}joint_2" multiplier="1" offset="-1.570796326794897" />
-   </joint>
-   <link name="${prefix}link_2_1">
+     <limit
+       lower="-6.2831853"
+       upper="6.2831853"
+       effort="100000"
+       velocity="${joint_6_vel_limit}" />
+  </joint>
+  <!-- <joint name="${prefix}joint_3" type="revolute">
+      <origin xyz="0 1.175 0.0955" rpy="3.1416 0 3.1416" />
+      <parent link="${prefix}link_2" />
+      <child link="${prefix}link_3" />
+      <axis xyz="0 0 -1" />
+      <limit
+        lower="-6.2831853"
+        upper="6.2831853"
+        effort="0"
+        velocity="${joint_3_vel_limit}" />
+  </joint> -->
+  <!-- <link name="${prefix}link_2_2">
+   <inertial>
+     <origin xyz="0 0 0" rpy="0 0 0" />
+     <mass value="0.01" />
+     <inertia
+       ixx="0.00001"
+       ixy="0.00000"
+       ixz="0.00000"
+       iyy="0.00001"
+       iyz="0.00000"
+       izz="0.00000" />
+   </inertial>
+  </link>
+  <joint name="${prefix}l3_to_l22" type="continuous">
+    <origin xyz="0.34867 -0.0305 -0.165" rpy="0 0 3.1416" />
+    <parent link="${prefix}link_3" />
+    <child link="${prefix}link_2_2" />
+    <axis xyz="0 0 1" />
+    <mimic joint="${prefix}joint_2" multiplier="1" offset="-1.570796326794897" />
+  </joint>
+  <link name="${prefix}link_2_2_virtual">
+   <inertial>
+     <origin xyz="0 0 0" rpy="0 0 0" />
+     <mass value="0.01" />
+     <inertia
+       ixx="0.00001"
+       ixy="0.00000"
+       ixz="0.00000"
+       iyy="0.00001"
+       iyz="0.00000"
+       izz="0.00000" />
+   </inertial>
+  </link>
+  <joint name="${prefix}l22_to_l22v" type="continuous">
+    <origin xyz="0 0 0" rpy="0 0 0" />
+    <parent link="${prefix}link_2_2" />
+    <child link="${prefix}link_2_2_virtual" />
+    <axis xyz="0 0 1" />
+    <mimic joint="${prefix}joint_3" multiplier="1" offset="-1.570796326794897" />
+  </joint>
+  <link name="${prefix}link_2_2_real">
+     <inertial>
+       <origin
+         xyz="0.064434 0.51885 0.014848"
+         rpy="0 0 0" />
+       <mass
+         value="60.719" />
+       <inertia
+         ixx="5.5799"
+         ixy="0.13804"
+         ixz="0.0007529"
+         iyy="0.14481"
+         iyz="-0.0028767"
+         izz="5.6722" />
+     </inertial>
+     <visual>
+       <origin
+         xyz="0 0 0"
+         rpy="0 0 0" />
+       <geometry>
+         <mesh
+           filename="package://nj_220_2_7_gazebo/meshes/link_2_2.STL" />
+       </geometry>
+       <material
+         name="">
+         <color
+           rgba="1 0 0 1" />
+       </material>
+     </visual>
+     <collision>
+       <origin
+         xyz="0 0 0"
+         rpy="0 0 0" />
+       <geometry>
+         <mesh
+           filename="package://nj_220_2_7_gazebo/meshes/link_2_2.STL" />
+       </geometry>
+     </collision>
+   </link>
+  <joint name="${prefix}l22v_to_l22r" type="fixed">
+    <origin xyz="0 -1.175 -0.015" rpy="0 0 0" />
+    <parent link="${prefix}link_2_2_virtual" />
+    <child link="${prefix}link_2_2_real" />
+    <axis xyz="0 0 0" />
+    <limit
+      lower="-6.2831853"
+      upper="6.2831853"
+      effort="0"
+      velocity="0" />
+  </joint>
+  <link name="${prefix}link_2_1">
+   <inertial>
+     <origin xyz="0 0 0" rpy="0 0 0" />
+     <mass value="0.01" />
+     <inertia
+       ixx="0.00001"
+       ixy="0.00000"
+       ixz="0.00000"
+       iyy="0.00001"
+       iyz="0.00000"
+       izz="0.00000" />
+   </inertial>
+  </link>
+  <joint name="${prefix}l22v_to_l21" type="continuous">
+    <origin xyz="0 -1.175 -0.015" rpy="0 0 -0.087266" />
+    <parent link="${prefix}link_2_2_virtual" />
+    <child link="${prefix}link_2_1" />
+    <axis xyz="0 0 -1" />
+    <mimic joint="${prefix}joint_3" multiplier="1" offset="0" />
+  </joint>
+  <link name="${prefix}link_2_1_virtual">
+   <inertial>
+     <origin xyz="0 0 0" rpy="0 0 0" />
+     <mass value="0.01" />
+     <inertia
+       ixx="0.00001"
+       ixy="0.00000"
+       ixz="0.00000"
+       iyy="0.00001"
+       iyz="0.00000"
+       izz="0.00000" />
+   </inertial>
+  </link>
+  <joint name="${prefix}l21_to_l21v" type="continuous">
+    <origin xyz="0 0 0" rpy="0 0 0" />
+    <parent link="${prefix}link_2_1" />
+    <child link="${prefix}link_2_1_virtual" />
+    <axis xyz="0 0 -1" />
+    <mimic joint="${prefix}joint_2" multiplier="1" offset="0" />
+  </joint>
+  <link name="${prefix}link_2_1_real">
      <inertial>
        <origin
@@ -444,88 +589,33 @@
      </collision>
    </link>
-   <joint name="${prefix}joint_2_1" type="continuous">
-     <origin
-       xyz="-0.4 0.499 -0.1945"
-       rpy="0 0 -0.087266" />
-     <parent
-       link="${prefix}link_1" />
-     <child
-       link="${prefix}link_2_1" />
-     <axis
-       xyz="0 0 -1" />
-     <mimic joint="${prefix}joint_3" multiplier="1" offset="0" />
-   </joint>
-   <link name="${prefix}link_2_2_virtual">
-     <inertial>
-       <origin xyz="0 0 0" rpy="0 0 0" />
-       <mass value="0.01" />
-       <inertia
-         ixx="0.00001"
-         ixy="0.00000"
-         ixz="0.00000"
-         iyy="0.00001"
-         iyz="0.00000"
-         izz="0.00000" />
-     </inertial>
-   </link>
-   <joint name="${prefix}joint_2_2" type="continuous">
-     <origin
-       xyz="0.35 0 0.015"
-       rpy="0 0 0.08723" />
-     <parent
-       link="${prefix}link_2_1" />
-     <child
-       link="${prefix}link_2_2_virtual" />
-     <axis
-       xyz="0 0 1" />
-     <mimic joint="${prefix}joint_3" multiplier="1" offset="0"/>
-   </joint>
-   <link name="${prefix}link_2_2">
-     <inertial>
-       <origin
-         xyz="0.064434 0.51885 0.014848"
-         rpy="0 0 0" />
-       <mass
-         value="60.719" />
-       <inertia
-         ixx="5.5799"
-         ixy="0.13804"
-         ixz="0.0007529"
-         iyy="0.14481"
-         iyz="-0.0028767"
-         izz="5.6722" />
-     </inertial>
-     <visual>
-       <origin
-         xyz="0 0 0"
-         rpy="0 0 0" />
-       <geometry>
-         <mesh
-           filename="package://nj_220_2_7_gazebo/meshes/link_2_2.STL" />
-       </geometry>
-       <material
-         name="">
-         <color
-           rgba="1 0 0 1" />
-       </material>
-     </visual>
-     <collision>
-       <origin
-         xyz="0 0 0"
-         rpy="0 0 0" />
-       <geometry>
-         <mesh
-           filename="package://nj_220_2_7_gazebo/meshes/link_2_2.STL" />
-       </geometry>
-     </collision>
-   </link>
-   <joint name="${prefix}joint_2_3" type="continuous">
-     <origin xyz="0.0 0.0 0.0" rpy="0 0 0" />
-     <parent link="${prefix}link_2_2_virtual" />
-     <child link="${prefix}link_2_2" />
-     <axis xyz="0 0 -1" />
-     <mimic joint="${prefix}joint_2" multiplier="-1" offset="0"/>
-   </joint>
- <!-- End Parallel Linkages -->
+  <joint name="${prefix}l21v_to_l21r" type="fixed">
+    <origin xyz="-0.35 0 -0.015" rpy="0 0 0" />
+    <parent link="${prefix}link_2_1_virtual" />
+    <child link="${prefix}link_2_1_real" />
+    <axis xyz="0 0 0" />
+    <limit
+      lower="-6.2831853"
+      upper="6.2831853"
+      effort="0"
+      velocity="0" />
+  </joint>
+  <gazebo>
+    <joint name="${prefix}closing_joint_1" type="revolute">
+      <parent>${prefix}link_1</parent>
+      <child>${prefix}link_2_1_real</child>
+      <pose relative_to="${prefix}link_1"> -0.4 0.499 -0.0955 0 0 -0.087266</pose>
+      <axis>
+        <xyz>0 0 1</xyz>
+      </axis>
+    </joint>
+    <joint name="${prefix}closing_joint_2" type="revolute">
+      <parent>${prefix}link_2_1_real</parent>
+      <child>${prefix}link_2</child>
+      <pose relative_to="${prefix}link_1"> 0 0 0.291 -3.142 0 -3.055</pose>
+      <axis>
+        <xyz>0 0 1</xyz>
+      </axis>
+    </joint>
+  </gazebo> -->
   <link name="${prefix}flange">
     <inertial>

File: nj_220_2_7_description/urdf/nj_220_2_7_gazebo.xacro (robot description, xacro)
@@ -11,5 +11,4 @@
     </plugin>
   </gazebo>
-  <!-- Mimic Joint Plug in for Gazebo-->
   <xacro:macro name="mimic_joint_plugin_gazebo" params="name_prefix parent_joint mimic_joint has_pid:=false multiplier:=1.0 offset:=0 sensitiveness:=0.0 max_effort:=1.0 robot_namespace:=''">
     <gazebo>
@@ -32,40 +31,5 @@
   <xacro:mimic_joint_plugin_gazebo name_prefix="${prefix}joint_2m"
     parent_joint="${prefix}joint_2" mimic_joint="${prefix}joint_2m"
-    has_pid="false" multiplier="1.0" max_effort="10000.0" />
-  <!--Mimic Joint Plug in for Gazebo -->
-  <!--Mimic Joint Plug in for Gazebo-->
-    <!-- <xacro:macro name="mimic_joint_plugin_gazebo" params="name_prefix parent_joint mimic_joint has_pid:=false multiplier:=1.0 offset:=0 sensitiveness:=0.0 max_effort:=1.0 robot_namespace:=''">
-      <gazebo>
-        <plugin name="${name_prefix}mimic_joint_plugin" filename="libroboticsgroup_gazebo_mimic_joint_plugin.so">
-          <joint>${parent_joint}</joint>
-          <mimicJoint>${mimic_joint}</mimicJoint>
-          <xacro:if value="${has_pid}">
-            <hasPID />
-          </xacro:if>
-          <multiplier>${multiplier}</multiplier>
-          <offset>${offset}</offset>
-          <sensitiveness>${sensitiveness}</sensitiveness>
-          <maxEffort>${max_effort}</maxEffort>
-          <xacro:unless value="${robot_namespace == ''}">
-            <robotNamespace>($robot_namespace)</robotNamespace>
-          </xacro:unless>
-        </plugin>
-      </gazebo>
-    </xacro:macro>
-    <xacro:macro name="controller_plugin_gazebo" params="robot_namespace:=''">
-      <gazebo>
-        <plugin name="ros_control" filename="libgazebo_ros_control.so">
-          <xacro:unless value="${robot_namespace == ''}">
-            <robotNamespace>($robot_namespace)</robotNamespace>
-          </xacro:unless>
-          <controlPeriod>0.001</controlPeriod>
-        </plugin>
-      </gazebo>
-    </xacro:macro>
-    <controller_plugin_gazebo />
-     <xacro:mimic_joint_plugin_gazebo name_prefix="${prefix}joint_2m"
-          parent_joint="${prefix}joint_2" mimic_joint="${prefix}joint_2m"
-          has_pid="false" multiplier="1.0" max_effort="10.0" /> -->
-      <!--Mimic Joint Plug in for Gazebo-->
+    has_pid="false" multiplier="-1.0" max_effort="10000.0" />
   <gazebo reference="${prefix}link_6_to_flange">
       <provideFeedback>true</provideFeedback>

Commit message: tried some methods but they don't work

File: nj_220_2_7_description/urdf/nj_220_2_7.xacro (robot description, xacro)
@@ -1,6 +1,6 @@
 <?xml version="1.0" ?>
 <robot xmlns:xacro="http://ros.org/wiki/xacro">
-<xacro:macro name="nj_220_2_7" params="prefix:='' interface:=hardware_interface/EffortJointInterface">
-<!-- <xacro:macro name="nj_220_2_7" params="prefix:='' interface:=hardware_interface/PositionJointInterface"> -->
+<!-- <xacro:macro name="nj_220_2_7" params="prefix:='' interface:=hardware_interface/EffortJointInterface"> -->
+<xacro:macro name="nj_220_2_7" params="prefix:='' interface:=hardware_interface/PositionJointInterface">
   <xacro:property name="joint_1_vel_limit" value="1.74533" />    <!--  100°/s -->
   <xacro:property name="joint_2_vel_limit" value="1.5708"  />    <!--  90°/s -->
@@ -9,7 +9,7 @@
   <xacro:property name="joint_5_vel_limit" value="2.26893" />    <!--  130°/s -->
   <xacro:property name="joint_6_vel_limit" value="3.40339" />    <!--  195°/s -->
-  <xacro:property name="joint_1_eff_limit" value="10000" />
-  <xacro:property name="joint_2_eff_limit" value="10000" />
-  <xacro:property name="joint_3_eff_limit" value="10000" />
+  <xacro:property name="joint_1_eff_limit" value="100000" />
+  <xacro:property name="joint_2_eff_limit" value="100000" />
+  <xacro:property name="joint_3_eff_limit" value="100000" />
   <xacro:property name="joint_4_eff_limit" value="1230" />
   <xacro:property name="joint_5_eff_limit" value="1230" />
@@ -398,9 +398,9 @@
    </link>
   <joint name="${prefix}joint_2m" type="revolute">
-     <origin xyz="0 1.175 0.0955" rpy="3.1416 0 -1.5708" />
+     <origin xyz="0 1.175 0.0955" rpy="3.1416 0 3.1416" />
      <parent link="${prefix}link_2" />
      <child link="${prefix}link_3_virtual" />
      <axis xyz="0 0 -1" />
-     <mimic joint="${prefix}joint_2" multiplier="1" offset="-1.570796326794897" />
+     <mimic joint="${prefix}joint_2" multiplier="1" offset="0" />
      <limit
        lower="-6.2831853"
@@ -420,5 +420,5 @@
         velocity="${joint_3_vel_limit}" />
   </joint> -->
-  <!-- <link name="${prefix}link_2_2">
+  <link name="${prefix}link_2_2">
    <inertial>
      <origin xyz="0 0 0" rpy="0 0 0" />
@@ -433,10 +433,15 @@
    </inertial>
   </link>
-  <joint name="${prefix}l3_to_l22" type="continuous">
-    <origin xyz="0.34867 -0.0305 -0.165" rpy="0 0 3.1416" />
+  <joint name="${prefix}l3_to_l22" type="revolute">
+    <origin xyz="0.34867 -0.0305 -0.165" rpy="0 0 1.570796326794897" />
     <parent link="${prefix}link_3" />
     <child link="${prefix}link_2_2" />
     <axis xyz="0 0 1" />
-    <mimic joint="${prefix}joint_2" multiplier="1" offset="-1.570796326794897" />
+    <mimic joint="${prefix}joint_2" multiplier="1" offset="0" />
+    <limit
+      lower="-6.2831853"
+      upper="6.2831853"
+      effort="${joint_6_eff_limit}"
+      velocity="${joint_6_vel_limit}" />
   </joint>
   <link name="${prefix}link_2_2_virtual">
@@ -453,10 +458,15 @@
    </inertial>
   </link>
-  <joint name="${prefix}l22_to_l22v" type="continuous">
-    <origin xyz="0 0 0" rpy="0 0 0" />
+  <joint name="${prefix}l22_to_l22v" type="revolute">
+    <origin xyz="0 0 0" rpy="0 0 -1.570796326794897" />
     <parent link="${prefix}link_2_2" />
     <child link="${prefix}link_2_2_virtual" />
     <axis xyz="0 0 1" />
-    <mimic joint="${prefix}joint_3" multiplier="1" offset="-1.570796326794897" />
+    <mimic joint="${prefix}joint_3" multiplier="1" offset="0" />
+    <limit
+      lower="-6.2831853"
+      upper="6.2831853"
+      effort="${joint_6_eff_limit}"
+      velocity="${joint_6_vel_limit}" />
   </joint>
   <link name="${prefix}link_2_2_real">
@@ -523,5 +533,5 @@
    </inertial>
   </link>
-  <joint name="${prefix}l22v_to_l21" type="continuous">
+  <joint name="${prefix}l22v_to_l21" type="revolute">
     <origin xyz="0 -1.175 -0.015" rpy="0 0 -0.087266" />
     <parent link="${prefix}link_2_2_virtual" />
@@ -529,4 +539,9 @@
     <axis xyz="0 0 -1" />
     <mimic joint="${prefix}joint_3" multiplier="1" offset="0" />
+    <limit
+      lower="-6.2831853"
+      upper="6.2831853"
+      effort="${joint_6_eff_limit}"
+      velocity="${joint_6_vel_limit}" />
   </joint>
   <link name="${prefix}link_2_1_virtual">
@@ -543,5 +558,5 @@
    </inertial>
   </link>
-  <joint name="${prefix}l21_to_l21v" type="continuous">
+  <joint name="${prefix}l21_to_l21v" type="revolute">
     <origin xyz="0 0 0" rpy="0 0 0" />
     <parent link="${prefix}link_2_1" />
@@ -549,4 +564,9 @@
     <axis xyz="0 0 -1" />
     <mimic joint="${prefix}joint_2" multiplier="1" offset="0" />
+    <limit
+      lower="-6.2831853"
+      upper="6.2831853"
+      effort="${joint_6_eff_limit}"
+      velocity="${joint_6_vel_limit}" />
   </joint>
   <link name="${prefix}link_2_1_real">
@@ -590,19 +610,19 @@
    </link>
   <joint name="${prefix}l21v_to_l21r" type="fixed">
-    <origin xyz="-0.35 0 -0.015" rpy="0 0 0" />
-    <parent link="${prefix}link_2_1_virtual" />
-    <child link="${prefix}link_2_1_real" />
-    <axis xyz="0 0 0" />
-    <limit
-      lower="-6.2831853"
-      upper="6.2831853"
-      effort="0"
-      velocity="0" />
-  </joint>
+     <origin xyz="-0.35 0 -0.015" rpy="0 0 0" />
+     <parent link="${prefix}link_2_1_virtual" />
+     <child link="${prefix}link_2_1_real" />
+     <axis xyz="0 0 0" />
+     <limit
+       lower="-6.2831853"
+       upper="6.2831853"
+       effort="0"
+       velocity="0" />
+   </joint>
   <gazebo>
     <joint name="${prefix}closing_joint_1" type="revolute">
       <parent>${prefix}link_1</parent>
       <child>${prefix}link_2_1_real</child>
-      <pose relative_to="${prefix}link_1"> -0.4 0.499 -0.0955 0 0 -0.087266</pose>
+      <pose relative_to="${prefix}link_1"> -0.400, 0.499, -0.195 -0.000, -0.000, -0.087</pose>
       <axis>
         <xyz>0 0 1</xyz>
@@ -612,10 +632,10 @@
       <parent>${prefix}link_2_1_real</parent>
       <child>${prefix}link_2</child>
-      <pose relative_to="${prefix}link_1"> 0 0 0.291 -3.142 0 -3.055</pose>
+      <pose relative_to="${prefix}link_2_1_real"> 0 0 0 0 0 0</pose>
       <axis>
         <xyz>0 0 1</xyz>
       </axis>
     </joint>
-  </gazebo> -->
+  </gazebo>
   <link name="${prefix}flange">
     <inertial>

File: nj_220_2_7_description/urdf/nj_220_2_7_gazebo.xacro (robot description, xacro)
@@ -11,25 +11,4 @@
     </plugin>
   </gazebo>
-  <xacro:macro name="mimic_joint_plugin_gazebo" params="name_prefix parent_joint mimic_joint has_pid:=false multiplier:=1.0 offset:=0 sensitiveness:=0.0 max_effort:=1.0 robot_namespace:=''">
-    <gazebo>
-      <plugin name="${name_prefix}mimic_joint_plugin" filename="libroboticsgroup_gazebo_mimic_joint_plugin.so">
-        <joint>${parent_joint}</joint>
-        <mimicJoint>${mimic_joint}</mimicJoint>
-        <xacro:if value="${has_pid}">
-          <hasPID />
-        </xacro:if>
-        <multiplier>${multiplier}</multiplier>
-        <offset>${offset}</offset>
-        <sensitiveness>${sensitiveness}</sensitiveness>
-        <maxEffort>${max_effort}</maxEffort>
-        <xacro:unless value="${robot_namespace == ''}">
-          <robotNamespace>($robot_namespace)</robotNamespace>
-        </xacro:unless>
-      </plugin>
-    </gazebo>
-  </xacro:macro>
-  <xacro:mimic_joint_plugin_gazebo name_prefix="${prefix}joint_2m"
-    parent_joint="${prefix}joint_2" mimic_joint="${prefix}joint_2m"
-    has_pid="false" multiplier="-1.0" max_effort="10000.0" />
   <gazebo reference="${prefix}link_6_to_flange">
       <provideFeedback>true</provideFeedback>

File: nj_220_2_7_description/urdf/nj_220_2_7_transmission.xacro (robot description, xacro)
@@ -20,4 +20,13 @@
     </actuator>
   </transmission>
+  <!-- <transmission name="${prefix}joint_2m_trans">
+   <type>transmission_interface/SimpleTransmission</type>
+   <joint name="${prefix}joint_2m">
+     <hardwareInterface>${interface}</hardwareInterface>
+   </joint>
+   <actuator name="${prefix}joint_2m_motor">
+     <mechanicalReduction>1</mechanicalReduction>
+   </actuator>
+ </transmission> -->
   <transmission name="${prefix}tran_3">
     <type>transmission_interface/SimpleTransmission</type>
