Commit message: Version with 2 urdf branch and gazebo link in joint 3

File: nj_220_2_7_description/urdf/nj_220_2_7.xacro (robot description, xacro)
@@ -522,8 +522,322 @@
     <axis xyz="0 0 0" />
   </joint>
+  <!-- Stroke Ends -->
+  <link name="${prefix}external_piece">
+    <inertial>
+      <origin
+        xyz="0.25149 0 0.08305"
+        rpy="0 0 0" />
+      <mass
+        value="11.17" />
+      <inertia
+        ixx="0.12505051"
+        ixy="0"
+        ixz="0.20615167"
+        iyy="0.86139689"
+        iyz="0"
+        izz="0.75193919" />
+    </inertial>
+    <visual>
+      <origin
+        xyz="0 0 0"
+        rpy="0 0 0" />
+      <geometry>
+        <mesh
+          filename="package://nj_220_2_7_gazebo/meshes/external_part.STL" />
+      </geometry>
+    </visual>
+    <collision>
+      <origin
+        xyz="0 0 0"
+        rpy="0 0 0" />
+      <geometry>
+        <mesh
+          filename="package://nj_220_2_7_gazebo/meshes/external_part.STL" />
+      </geometry>
+    </collision>
+  </link>
+  <joint name="${prefix}joint_external_piece" type="fixed">
+    <origin
+      xyz="0 0 0"
+      rpy="0 0 0" />
+    <parent
+      link="${prefix}link_1" />
+    <child
+      link="${prefix}external_piece" />
+    <axis xyz="0 0 0" />
+  </joint>
+  <link name="${prefix}motor_1">
+    <inertial>
+      <origin
+        xyz="0 0.00059 -0.13134"
+        rpy="0 0 0" />
+      <mass
+        value="74.18" />
+      <inertia
+        ixx="2.03862179"
+        ixy="0.00000294"
+        ixz="0.00001194"
+        iyy="2.03393681"
+        iyz="-0.01109897"
+        izz="0.37378121" />
+    </inertial>
+    <visual>
+      <origin
+        xyz="0 0 0"
+        rpy="0 0 0" />
+      <geometry>
+        <mesh
+          filename="package://nj_220_2_7_gazebo/meshes/motor_80.STL" />
+      </geometry>
+    </visual>
+    <collision>
+      <origin
+        xyz="0 0 0"
+        rpy="0 0 0" />
+      <geometry>
+        <mesh
+          filename="package://nj_220_2_7_gazebo/meshes/motor_80.STL" />
+      </geometry>
+    </collision>
+  </link>
+  <joint name="${prefix}joint_motor_1" type="fixed">
+    <origin
+      xyz="-0.1567 0.0905 0.12075"
+      rpy="0 0 4.194026193" />
+    <parent
+      link="${prefix}link_1" />
+    <child
+      link="${prefix}motor_1" />
+    <axis xyz="0 0 0" />
+  </joint>
+  <link name="${prefix}motor_2">
+    <inertial>
+      <origin
+        xyz="0 0.00055 -0.14385"
+        rpy="0 0 0" />
+      <mass
+        value="80.26" />
+      <inertia
+        ixx="2.5764983"
+        ixy="0.00000380"
+        ixz="0.01312758"
+        iyy="2.49873445"
+        iyz="-0.0000105"
+        izz="0.40399789" />
+    </inertial>
+    <visual>
+      <origin
+        xyz="0 0 0"
+        rpy="0 0 0" />
+      <geometry>
+        <mesh
+          filename="package://nj_220_2_7_gazebo/meshes/motor_90.STL" />
+      </geometry>
+    </visual>
+    <collision>
+      <origin
+        xyz="0 0 0"
+        rpy="0 0 0" />
+      <geometry>
+        <mesh
+          filename="package://nj_220_2_7_gazebo/meshes/motor_90.STL" />
+      </geometry>
+    </collision>
+  </link>
+  <joint name="${prefix}joint_motor_2" type="fixed">
+    <origin
+      xyz="0.400 0.2955 0.499"
+      rpy="-1.570796327 1.570796327 0" />
+    <parent
+      link="${prefix}link_1" />
+    <child
+      link="${prefix}motor_2" />
+      <axis xyz="0 0 0" />
+  </joint>
+  <link name="${prefix}motor_3">
+    <inertial>
+      <origin
+        xyz="0 0.00059 -0.13134"
+        rpy="0 0 0" />
+      <mass
+        value="74.18" />
+      <inertia
+        ixx="2.03862179"
+        ixy="0.00000294"
+        ixz="0.00001194"
+        iyy="2.03393681"
+        iyz="-0.01109897"
+        izz="0.37378121" />
+    </inertial>
+    <visual>
+      <origin
+        xyz="0 0 0"
+        rpy="0 0 0" />
+      <geometry>
+        <mesh
+          filename="package://nj_220_2_7_gazebo/meshes/motor_80.STL" />
+      </geometry>
+    </visual>
+    <collision>
+      <origin
+        xyz="0 0 0"
+        rpy="0 0 0" />
+      <geometry>
+        <mesh
+          filename="package://nj_220_2_7_gazebo/meshes/motor_80.STL" />
+      </geometry>
+    </collision>
+  </link>
+  <joint name="${prefix}joint_motor_3" type="fixed">
+    <origin
+      xyz="0.400 -0.358 0.499"
+      rpy="1.570796327 1.570796327 0" />
+    <parent
+      link="${prefix}link_1" />
+    <child
+      link="${prefix}motor_3" />
+      <axis xyz="0 0 0" />
+  </joint>
+  <link name="${prefix}motor_4">
+    <inertial>
+      <origin
+        xyz="0.00125 0 -0.0852"
+        rpy="0 0 0" />
+      <mass
+        value="28" />
+      <inertia
+        ixx="0.33783188"
+        ixy="-0.00000254"
+        ixz="-0.00532880"
+        iyy="0.34073438"
+        iyz="0.00000366"
+        izz="0.08086422" />
+    </inertial>
+    <visual>
+      <origin
+        xyz="0 0 0"
+        rpy="0 0 0" />
+      <geometry>
+        <mesh
+          filename="package://nj_220_2_7_gazebo/meshes/motor_50.STL" />
+      </geometry>
+    </visual>
+    <collision>
+      <origin
+        xyz="0 0 0"
+        rpy="0 0 0" />
+      <geometry>
+        <mesh
+          filename="package://nj_220_2_7_gazebo/meshes/motor_50.STL" />
+      </geometry>
+    </collision>
+  </link>
+  <joint name="${prefix}joint_motor_4"
+    type="fixed">
+    <origin
+      xyz="-0.200 0.21052 0.175"
+      rpy="3.141592654 1.570796327 0" />
+    <parent
+      link="${prefix}link_3" />
+    <child
+      link="${prefix}motor_4" />
+    <axis
+      xyz="0 -1 0" />
+  </joint>
+  <link name="${prefix}motor_5">
+    <inertial>
+      <origin
+        xyz="0.00125 0 -0.0852"
+        rpy="0 0 0" />
+      <mass
+        value="28" />
+      <inertia
+        ixx="0.33783188"
+        ixy="-0.00000254"
+        ixz="-0.00532880"
+        iyy="0.34073438"
+        iyz="0.00000366"
+        izz="0.08086422" />
+    </inertial>
+    <visual>
+      <origin
+        xyz="0 0 0"
+        rpy="0 0 0" />
+      <geometry>
+        <mesh
+          filename="package://nj_220_2_7_gazebo/meshes/motor_50.STL" />
+      </geometry>
+    </visual>
+    <collision>
+      <origin
+        xyz="0 0 0"
+        rpy="0 0 0" />
+      <geometry>
+        <mesh
+          filename="package://nj_220_2_7_gazebo/meshes/motor_50.STL" />
+      </geometry>
+    </collision>
+  </link>
+  <joint name="${prefix}joint_motor_5"
+    type="fixed">
+    <origin
+      xyz="-0.1675 0 0.250"
+      rpy="1.570796327 0 -1.570796327" />
+    <parent
+      link="${prefix}link_3" />
+    <child
+      link="${prefix}motor_5" />
+    <axis
+      xyz="0 -1 0" />
+  </joint>
+  <link name="${prefix}motor_6">
+    <inertial>
+      <origin
+        xyz="0.00125 0 -0.0852"
+        rpy="0 0 0" />
+      <mass
+        value="28" />
+      <inertia
+        ixx="0.33783188"
+        ixy="-0.00000254"
+        ixz="-0.00532880"
+        iyy="0.34073438"
+        iyz="0.00000366"
+        izz="0.08086422" />
+    </inertial>
+    <visual>
+      <origin
+        xyz="0 0 0"
+        rpy="0 0 0" />
+      <geometry>
+        <mesh
+          filename="package://nj_220_2_7_gazebo/meshes/motor_50.STL" />
+      </geometry>
+    </visual>
+    <collision>
+      <origin
+        xyz="0 0 0"
+        rpy="0 0 0" />
+      <geometry>
+        <mesh
+          filename="package://nj_220_2_7_gazebo/meshes/motor_50.STL" />
+      </geometry>
+    </collision>
+  </link>
+  <joint name="${prefix}joint_motor_6"
+    type="fixed">
+    <origin
+      xyz="-0.1675 0.155 0.34577"
+      rpy="-1.570796327 0 1.570796327" />
+    <parent
+      link="${prefix}link_3" />
+    <child
+      link="${prefix}motor_6" />
+    <axis
+      xyz="0 -1 0" />
+  </joint>
+  <!-- End Stroke End -->
 <xacro:include filename="$(find nj_220_2_7_description)/urdf/nj_220_2_7_transmission.xacro" />
 <xacro:nj_220_2_7_transmission prefix="${prefix}" interface="${interface}"/>
-<xacro:include filename="$(find nj_220_2_7_description)/urdf/nj_220_2_7_gazebo.xacro" />
-<xacro:nj_220_2_7_roscontrol prefix="${prefix}"/>
 </xacro:macro>
 </robot>

File: nj_220_2_7_gazebo/urdf/nj_220_2_7.xacro (robot description, xacro)
@@ -3,4 +3,8 @@
 <!-- <xacro:macro name="nj_220_2_7" params="prefix:='' interface:=hardware_interface/EffortJointInterface"> -->
 <xacro:macro name="nj_220_2_7" params="prefix:='' interface:=hardware_interface/PositionJointInterface">
+  <selfCollide>0</selfCollide>
+  <gazebo>
+    <selfCollide>0</selfCollide>
+  </gazebo>
   <xacro:property name="joint_1_vel_limit" value="1.74533" />    <!--  100°/s -->
   <xacro:property name="joint_2_vel_limit" value="1.5708"  />    <!--  90°/s -->
@@ -248,5 +252,5 @@
      </collision>
   </link>
-  <joint name="${prefix}joint_2_1" type="continuous">
+  <joint name="${prefix}joint_2_1" type="revolute">
     <origin
       xyz="0.350 0 0.015"
@@ -258,4 +262,9 @@
     <axis
       xyz="0 0 1" />
+    <limit
+      lower="-6.2831853"
+      upper="6.2831853"
+      effort="${joint_6_eff_limit}"
+      velocity="${joint_6_vel_limit}" />
   </joint>
   <link name="${prefix}link_2_3">
@@ -272,9 +281,14 @@
     </inertial>
   </link>
-  <joint name="${prefix}joint_2_2" type="continuous">
-    <origin xyz="0.0 1.175 0.0" rpy="0 0 0" />
+  <joint name="${prefix}joint_2_2" type="revolute">
+    <origin xyz="0.0 1.175 0.0" rpy="0 0 -0.087266" />
     <parent link="${prefix}link_2_2" />
     <child link="${prefix}link_2_3" />
     <axis xyz="0 0 1" />
+    <limit
+      lower="-6.2831853"
+      upper="6.2831853"
+      effort="${joint_6_eff_limit}"
+      velocity="${joint_6_vel_limit}" />
   </joint>
   <link name="${prefix}link_3">
@@ -317,15 +331,4 @@
     </collision>
   </link>
-  <joint name="${prefix}joint_3_1" type="continuous">
-    <origin
-      xyz="-0.34867 0.0305 0.1795"
-      rpy="1.571 0.000 -3.141" />
-    <parent
-      link="${prefix}link_2_3" />
-    <child
-      link="${prefix}link_3" />
-    <axis
-      xyz="0 0 1" />
-  </joint>
   <link name="${prefix}link_4">
     <inertial>
@@ -493,6 +496,48 @@
       velocity="${joint_6_vel_limit}" />
   </joint>
+  <joint name="${prefix}closing_joint" type="revolute">
+    <origin
+      xyz="0 0 1.175"
+      rpy="0 0 0" />
+    <parent
+      link="${prefix}link_2" />
+    <child
+      link="${prefix}link_3" />
+    <axis
+      xyz="0 1 0" />
+    <limit
+      lower="-6.2831853"
+      upper="6.2831853"
+      effort="${joint_6_eff_limit}"
+      velocity="${joint_6_vel_limit}" />
+  </joint>
   <gazebo>
-    <joint name="${prefix}closing_joint" type="continuous">
+    <joint name="${prefix}joint_3_1" type="fixed">
+      <parent>${prefix}link_2_3</parent>
+      <child>${prefix}link_3</child>
+      <pose relative_to="${prefix}link_2"> -0.350, 0, 0.179, 1.571, 0, -3.054326654</pose>
+      <axis>
+        <xyz>0 0 1</xyz>
+      </axis>
+    </joint>
+  </gazebo>
+  <!-- <joint name="${prefix}joint_3_1" type="fixed">
+    <origin
+      xyz="-0.350 0 0.179"
+      rpy="1.571 0.000 -3.054326654" />
+    <parent
+      link="${prefix}link_2_3" />
+    <child
+      link="${prefix}link_3" />
+    <axis
+      xyz="0 0 1" />
+    <limit
+      lower="-6.2831853"
+      upper="6.2831853"
+      effort="${joint_6_eff_limit}"
+      velocity="${joint_6_vel_limit}" />
+  </joint> -->
+  <!-- <gazebo>
+    <joint name="${prefix}closing_joint" type="revolute">
       <parent>${prefix}link_2</parent>
       <child>${prefix}link_3</child>
@@ -502,5 +547,5 @@
       </axis>
     </joint>
-  </gazebo>
+  </gazebo> -->
   <link name="${prefix}flange">
     <inertial>
@@ -522,7 +567,323 @@
     <axis xyz="0 0 0" />
   </joint>
-<xacro:include filename="$(find nj_220_2_7_description)/urdf/nj_220_2_7_transmission.xacro" />
+  <!-- Stroke Ends -->
+  <link name="${prefix}external_piece">
+    <inertial>
+      <origin
+        xyz="0.25149 0 0.08305"
+        rpy="0 0 0" />
+      <mass
+        value="11.17" />
+      <inertia
+        ixx="0.12505051"
+        ixy="0"
+        ixz="0.20615167"
+        iyy="0.86139689"
+        iyz="0"
+        izz="0.75193919" />
+    </inertial>
+    <visual>
+      <origin
+        xyz="0 0 0"
+        rpy="0 0 0" />
+      <geometry>
+        <mesh
+          filename="package://nj_220_2_7_gazebo/meshes/external_part.STL" />
+      </geometry>
+    </visual>
+    <collision>
+      <origin
+        xyz="0 0 0"
+        rpy="0 0 0" />
+      <geometry>
+        <mesh
+          filename="package://nj_220_2_7_gazebo/meshes/external_part.STL" />
+      </geometry>
+    </collision>
+  </link>
+  <joint name="${prefix}joint_external_piece" type="fixed">
+    <origin
+      xyz="0 0 0"
+      rpy="0 0 0" />
+    <parent
+      link="${prefix}link_1" />
+    <child
+      link="${prefix}external_piece" />
+    <axis xyz="0 0 0" />
+  </joint>
+  <link name="${prefix}motor_1">
+    <inertial>
+      <origin
+        xyz="0 0.00059 -0.13134"
+        rpy="0 0 0" />
+      <mass
+        value="74.18" />
+      <inertia
+        ixx="2.03862179"
+        ixy="0.00000294"
+        ixz="0.00001194"
+        iyy="2.03393681"
+        iyz="-0.01109897"
+        izz="0.37378121" />
+    </inertial>
+    <visual>
+      <origin
+        xyz="0 0 0"
+        rpy="0 0 0" />
+      <geometry>
+        <mesh
+          filename="package://nj_220_2_7_gazebo/meshes/motor_80.STL" />
+      </geometry>
+    </visual>
+    <collision>
+      <origin
+        xyz="0 0 0"
+        rpy="0 0 0" />
+      <geometry>
+        <mesh
+          filename="package://nj_220_2_7_gazebo/meshes/motor_80.STL" />
+      </geometry>
+    </collision>
+  </link>
+  <joint name="${prefix}joint_motor_1" type="fixed">
+    <origin
+      xyz="-0.1567 0.0905 0.12075"
+      rpy="0 0 4.194026193" />
+    <parent
+      link="${prefix}link_1" />
+    <child
+      link="${prefix}motor_1" />
+    <axis xyz="0 0 0" />
+  </joint>
+  <link name="${prefix}motor_2">
+    <inertial>
+      <origin
+        xyz="0 0.00055 -0.14385"
+        rpy="0 0 0" />
+      <mass
+        value="80.26" />
+      <inertia
+        ixx="2.5764983"
+        ixy="0.00000380"
+        ixz="0.01312758"
+        iyy="2.49873445"
+        iyz="-0.0000105"
+        izz="0.40399789" />
+    </inertial>
+    <visual>
+      <origin
+        xyz="0 0 0"
+        rpy="0 0 0" />
+      <geometry>
+        <mesh
+          filename="package://nj_220_2_7_gazebo/meshes/motor_90.STL" />
+      </geometry>
+    </visual>
+    <collision>
+      <origin
+        xyz="0 0 0"
+        rpy="0 0 0" />
+      <geometry>
+        <mesh
+          filename="package://nj_220_2_7_gazebo/meshes/motor_90.STL" />
+      </geometry>
+    </collision>
+  </link>
+  <joint name="${prefix}joint_motor_2" type="fixed">
+    <origin
+      xyz="0.400 0.2955 0.499"
+      rpy="-1.570796327 1.570796327 0" />
+    <parent
+      link="${prefix}link_1" />
+    <child
+      link="${prefix}motor_2" />
+      <axis xyz="0 0 0" />
+  </joint>
+  <link name="${prefix}motor_3">
+    <inertial>
+      <origin
+        xyz="0 0.00059 -0.13134"
+        rpy="0 0 0" />
+      <mass
+        value="74.18" />
+      <inertia
+        ixx="2.03862179"
+        ixy="0.00000294"
+        ixz="0.00001194"
+        iyy="2.03393681"
+        iyz="-0.01109897"
+        izz="0.37378121" />
+    </inertial>
+    <visual>
+      <origin
+        xyz="0 0 0"
+        rpy="0 0 0" />
+      <geometry>
+        <mesh
+          filename="package://nj_220_2_7_gazebo/meshes/motor_80.STL" />
+      </geometry>
+    </visual>
+    <collision>
+      <origin
+        xyz="0 0 0"
+        rpy="0 0 0" />
+      <geometry>
+        <mesh
+          filename="package://nj_220_2_7_gazebo/meshes/motor_80.STL" />
+      </geometry>
+    </collision>
+  </link>
+  <joint name="${prefix}joint_motor_3" type="fixed">
+    <origin
+      xyz="0.400 -0.358 0.499"
+      rpy="1.570796327 1.570796327 0" />
+    <parent
+      link="${prefix}link_1" />
+    <child
+      link="${prefix}motor_3" />
+      <axis xyz="0 0 0" />
+  </joint>
+  <link name="${prefix}motor_4">
+    <inertial>
+      <origin
+        xyz="0.00125 0 -0.0852"
+        rpy="0 0 0" />
+      <mass
+        value="28" />
+      <inertia
+        ixx="0.33783188"
+        ixy="-0.00000254"
+        ixz="-0.00532880"
+        iyy="0.34073438"
+        iyz="0.00000366"
+        izz="0.08086422" />
+    </inertial>
+    <visual>
+      <origin
+        xyz="0 0 0"
+        rpy="0 0 0" />
+      <geometry>
+        <mesh
+          filename="package://nj_220_2_7_gazebo/meshes/motor_50.STL" />
+      </geometry>
+    </visual>
+    <collision>
+      <origin
+        xyz="0 0 0"
+        rpy="0 0 0" />
+      <geometry>
+        <mesh
+          filename="package://nj_220_2_7_gazebo/meshes/motor_50.STL" />
+      </geometry>
+    </collision>
+  </link>
+  <joint name="${prefix}joint_motor_4"
+    type="fixed">
+    <origin
+      xyz="-0.200 0.21052 0.175"
+      rpy="3.141592654 1.570796327 0" />
+    <parent
+      link="${prefix}link_3" />
+    <child
+      link="${prefix}motor_4" />
+    <axis
+      xyz="0 -1 0" />
+  </joint>
+  <link name="${prefix}motor_5">
+    <inertial>
+      <origin
+        xyz="0.00125 0 -0.0852"
+        rpy="0 0 0" />
+      <mass
+        value="28" />
+      <inertia
+        ixx="0.33783188"
+        ixy="-0.00000254"
+        ixz="-0.00532880"
+        iyy="0.34073438"
+        iyz="0.00000366"
+        izz="0.08086422" />
+    </inertial>
+    <visual>
+      <origin
+        xyz="0 0 0"
+        rpy="0 0 0" />
+      <geometry>
+        <mesh
+          filename="package://nj_220_2_7_gazebo/meshes/motor_50.STL" />
+      </geometry>
+    </visual>
+    <collision>
+      <origin
+        xyz="0 0 0"
+        rpy="0 0 0" />
+      <geometry>
+        <mesh
+          filename="package://nj_220_2_7_gazebo/meshes/motor_50.STL" />
+      </geometry>
+    </collision>
+  </link>
+  <joint name="${prefix}joint_motor_5"
+    type="fixed">
+    <origin
+      xyz="-0.1675 0 0.250"
+      rpy="1.570796327 0 -1.570796327" />
+    <parent
+      link="${prefix}link_3" />
+    <child
+      link="${prefix}motor_5" />
+    <axis
+      xyz="0 -1 0" />
+  </joint>
+  <link name="${prefix}motor_6">
+    <inertial>
+      <origin
+        xyz="0.00125 0 -0.0852"
+        rpy="0 0 0" />
+      <mass
+        value="28" />
+      <inertia
+        ixx="0.33783188"
+        ixy="-0.00000254"
+        ixz="-0.00532880"
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
File: nj_220_2_7_gazebo/urdf/nj_220_2_7_gazebo.xacro (robot description, xacro)
@@ -23,4 +23,64 @@
       </plugin>
   </gazebo>
+  <!-- <gazebo reference="nj_220_2_7">
+    <gravity>true</gravity>
+    <selfCollide>false</selfCollide>
+    <material>Gazebo/DarkGrey</material>
+  </gazebo> -->
+  <gazebo reference="${prefix}base_link">
+    <gravity>true</gravity>
+    <selfCollide>0</selfCollide>
+    <material>Gazebo/DarkGrey</material>
+  </gazebo>
+  <gazebo reference="${prefix}link_1">
+    <gravity>true</gravity>
+    <selfCollide>0</selfCollide>
+    <material>Gazebo/Grey</material>
+  </gazebo>
+  <gazebo reference="${prefix}link_2">
+    <gravity>true</gravity>
+    <selfCollide>0</selfCollide>
+    <material>Gazebo/Grey</material>
+  </gazebo>
+  <gazebo reference="${prefix}link_2_1">
+    <gravity>true</gravity>
+    <selfCollide>0</selfCollide>
+    <material>Gazebo/Grey</material>
+  </gazebo>
+  <gazebo reference="${prefix}link_2_2">
+    <gravity>true</gravity>
+    <selfCollide>0</selfCollide>
+    <material>Gazebo/Grey</material>
+  </gazebo>
+  <gazebo reference="${prefix}link_2_3">
+    <gravity>true</gravity>
+    <selfCollide>0</selfCollide>
+    <material>Gazebo/Grey</material>
+  </gazebo>
+  <gazebo reference="${prefix}link_3_virtual">
+    <gravity>true</gravity>
+    <selfCollide>0</selfCollide>
+    <material>Gazebo/Grey</material>
+  </gazebo>
+  <gazebo reference="${prefix}link_3">
+    <gravity>true</gravity>
+    <selfCollide>0</selfCollide>
+    <material>Gazebo/Grey</material>
+  </gazebo>
+  <gazebo reference="${prefix}link_4">
+    <gravity>true</gravity>
+    <selfCollide>0</selfCollide>
+    <material>Gazebo/Grey</material>
+  </gazebo>
+  <gazebo reference="${prefix}link_5">
+    <gravity>true</gravity>
+    <selfCollide>0</selfCollide>
+    <material>Gazebo/DarkGrey</material>
+  </gazebo>
+  <gazebo reference="${prefix}link_6">
+    <gravity>true</gravity>
+    <selfCollide>0</selfCollide>
+    <material>Gazebo/Black</material>
+  </gazebo>
 </xacro:macro>
 </robot>
