Commit message: Version with 2 urdf branch and gazebo link in joint 3

File: nj_220_2_7_moveit_config/config/gazebo_nj_220_2_7.urdf (robot description, URDF)
Before this commit: robot nj_220_2_7, 13 links, 12 joints
Links:
- added link external_piece, mass 11.17; collision mesh filename=package://nj_220_2_7_gazebo/meshes/external_part.STL; visual mesh filename=package://nj_220_2_7_gazebo/meshes/external_part.STL
- added link motor_1, mass 74.18; collision mesh filename=package://nj_220_2_7_gazebo/meshes/motor_80.STL; visual mesh filename=package://nj_220_2_7_gazebo/meshes/motor_80.STL
- added link motor_2, mass 80.26; collision mesh filename=package://nj_220_2_7_gazebo/meshes/motor_90.STL; visual mesh filename=package://nj_220_2_7_gazebo/meshes/motor_90.STL
- added link motor_3, mass 74.18; collision mesh filename=package://nj_220_2_7_gazebo/meshes/motor_80.STL; visual mesh filename=package://nj_220_2_7_gazebo/meshes/motor_80.STL
- added link motor_4, mass 28; collision mesh filename=package://nj_220_2_7_gazebo/meshes/motor_50.STL; visual mesh filename=package://nj_220_2_7_gazebo/meshes/motor_50.STL
- added link motor_5, mass 28; collision mesh filename=package://nj_220_2_7_gazebo/meshes/motor_50.STL; visual mesh filename=package://nj_220_2_7_gazebo/meshes/motor_50.STL
- added link motor_6, mass 28; collision mesh filename=package://nj_220_2_7_gazebo/meshes/motor_50.STL; visual mesh filename=package://nj_220_2_7_gazebo/meshes/motor_50.STL
- link link_1: mass 660.35 -> 120.57
- link link_2_2: mass 60.719 -> 60.72
- link link_3: mass 387.8 -> 303.81
Joints:
- added joint joint_external_piece: type fixed, parent link_1, child external_piece, origin xyz=0 0 0 rpy=0 0 0, axis 0 0 0
- added joint joint_motor_1: type fixed, parent link_1, child motor_1, origin xyz=-0.1567 0.0905 0.12075 rpy=0 0 4.194026193, axis 0 0 0
- added joint joint_motor_2: type fixed, parent link_1, child motor_2, origin xyz=0.400 0.2955 0.499 rpy=-1.570796327 1.570796327 0, axis 0 0 0
- added joint joint_motor_3: type fixed, parent link_1, child motor_3, origin xyz=0.400 -0.358 0.499 rpy=1.570796327 1.570796327 0, axis 0 0 0
- added joint joint_motor_4: type fixed, parent link_3, child motor_4, origin xyz=-0.200 0.21052 0.175 rpy=3.141592654 1.570796327 0, axis 0 -1 0
- added joint joint_motor_5: type fixed, parent link_3, child motor_5, origin xyz=-0.1675 0 0.250 rpy=1.570796327 0 -1.570796327, axis 0 -1 0
- added joint joint_motor_6: type fixed, parent link_3, child motor_6, origin xyz=-0.1675 0.155 0.34577 rpy=-1.570796327 0 1.570796327, axis 0 -1 0
- joint joint_1: axis 0 1 0 -> 0 0 1; limit lower=-1.570796327 upper=1.570796327 effort=10000 velocity=1.74533 -> lower=-1.570796327 upper=1.570796327 effort=100000 velocity=1.74533; origin xyz=0 0 0.331 rpy=1.570796327 0 0 -> xyz=0 0 0.331 rpy=0 0 0
- joint joint_2: axis 0 0 -1 -> 0 1 0; limit lower=-1.308996939 upper=1.658062789 effort=10000 velocity=1.5708 -> lower=-1.308996939 upper=1.658062789 effort=100000 velocity=1.5708; origin xyz=-0.4 0.499 0.0955 rpy=3.1416 0 -3.1416 -> xyz=0.4 0 0.499 rpy=0 0 0
- joint joint_2_1: axis 0 0 -1 -> 0 0 1; limit (none) -> lower=-6.2831853 upper=6.2831853 effort=0 velocity=0; mimic joint=joint_3 multiplier=1 offset=0 -> joint=joint_3 multiplier=-1 offset=0; origin xyz=-0.4 0.499 -0.1945 rpy=0 0 -0.087266 -> xyz=0.400 -0.1945 0.499 rpy=1.570796327 0.087266 3.141592654; type continuous -> revolute
- joint joint_2_2: origin xyz=0.35 0 0.015 rpy=0 0 0.08723 -> xyz=0.350 0 0.015 rpy=0 0 0.087266
- joint joint_2_3: axis 0 0 -1 -> 0 0 1; mimic joint=joint_2 multiplier=-1 offset=0 -> joint=joint_2 multiplier=1 offset=0
- joint joint_2m: axis 0 0 -1 -> 0 1 0; limit (none) -> lower=-6.2831853 upper=6.2831853 effort=100000 velocity=3.40339; mimic joint=joint_2 multiplier=1 offset=-1.570796326794897 -> joint=joint_2 multiplier=-1 offset=0; origin xyz=0 1.175 0.0955 rpy=3.1416 0 -1.5708 -> xyz=0 0 1.175 rpy=0 0 0; type continuous -> revolute
- joint joint_3: axis 0 0 -1 -> 0 -1 0; limit lower=-4.468042885 upper=0.174532925 effort=10000 velocity=1.91986 -> lower=-4.468042885 upper=0.174532925 effort=100000 velocity=1.91986
- joint joint_4: axis 0 0 1 -> 1 0 0; origin xyz=-0.105 0.25 0 rpy=-1.5708 -0.045821 1.5708 -> xyz=0.105 0 0.25 rpy=0 0 0
- joint joint_5: origin xyz=0 -0.128 1.0233 rpy=0 1.5708 0 -> xyz=1.02033 0 0 rpy=0 0 0
- joint joint_6: axis -1 0 0 -> 1 0 0; origin xyz=-0.2055 0.128 0 rpy=-0.045821 0 0 -> xyz=0.2085 0 0 rpy=0 0 0
- joint link_6_to_flange: origin xyz=0 0 -0.0395 rpy=3.1416 0 -1.5708 -> xyz=0 0 -0.0395 rpy=0 0 0

Commit message: merged gazebo and description urdf, need to fix some problem

File: nj_220_2_7_description/urdf/nj_220_2_7.xacro (robot description, xacro)
@@ -1,6 +1,6 @@
 <?xml version="1.0" ?>
 <robot xmlns:xacro="http://ros.org/wiki/xacro">
-<!-- <xacro:macro name="nj_220_2_7" params="prefix:='' interface:=hardware_interface/EffortJointInterface"> -->
-<xacro:macro name="nj_220_2_7" params="prefix:='' interface:=hardware_interface/PositionJointInterface">
+<!-- <xacro:macro name="nj_220_2_7" params="prefix:='' interface:=hardware_interface/EffortJointInterface type:=urdf"> -->
+  <xacro:macro name="nj_220_2_7" params="prefix:='' interface:=hardware_interface/PositionJointInterface type:=urdf">
   <xacro:property name="joint_1_vel_limit" value="1.74533" />    <!--  100°/s -->
   <xacro:property name="joint_2_vel_limit" value="1.5708"  />    <!--  90°/s -->
@@ -164,59 +164,139 @@
       velocity="${joint_2_vel_limit}" />
   </joint>
-  <link name="${prefix}link_3">
-    <inertial>
-      <origin
-        xyz="-0.04239 0.01939 0.2104"
-        rpy="0 0 0" />
-      <mass
-        value="303.81" />
-      <inertia
-        ixx="24.45402173"
-        ixy="-0.58037596"
-        ixz="-2.46563321"
-        iyy="20.71802091"
-        iyz="2.40454026"
-        izz="9.01610712" />
-    </inertial>
-    <visual>
-      <origin
-        xyz="0 0 0"
-        rpy="0 0 0" />
-      <geometry>
-        <mesh
-          filename="package://nj_220_2_7_gazebo/meshes/link_3.STL" />
-      </geometry>
-      <material
-        name="">
-        <color
-          rgba="1 0 0 1" />
-      </material>
-    </visual>
-    <collision>
-      <origin
-        xyz="0 0 0"
-        rpy="0 0 0" />
-      <geometry>
-        <mesh
-          filename="package://nj_220_2_7_gazebo/meshes/link_3.STL" />
-      </geometry>
-    </collision>
-  </link>
-  <joint name="${prefix}joint_3" type="revolute">
-    <origin
-      xyz="0 0 0"
-      rpy="0 0 0" />
-    <parent
-      link="${prefix}link_3_virtual" />
-    <child
-      link="${prefix}link_3" />
-    <axis
-      xyz="0 -1 0" />
-    <limit
-      lower="-4.468042885"
-      upper="0.174532925"
-      effort="${joint_3_eff_limit}"
-      velocity="${joint_3_vel_limit}" />
-  </joint>
+  <xacro:if value="${type == 'urdf'}">
+    <link name="${prefix}link_3_virtual">
+      <inertial>
+        <origin xyz="0 0 0" rpy="0 0 0" />
+        <mass value="0.01" />
+        <inertia
+          ixx="0.00001"
+          ixy="0.00000"
+          ixz="0.00000"
+          iyy="0.00001"
+          iyz="0.00000"
+          izz="0.00000" />
+      </inertial>
+    </link>
+    <joint name="${prefix}joint_2m" type="revolute">
+       <origin xyz="0 0 1.175" rpy="0 0 0" />
+       <parent link="${prefix}link_2" />
+       <child link="${prefix}link_3_virtual" />
+       <axis xyz="0 1 0" />
+       <mimic joint="${prefix}joint_2" multiplier="-1" offset="0" />
+       <limit
+         lower="-6.2831853"
+         upper="6.2831853"
+         effort="100000"
+         velocity="${joint_6_vel_limit}" />
+    </joint>
+    <link name="${prefix}link_3">
+      <inertial>
+        <origin
+          xyz="-0.04239 0.01939 0.2104"
+          rpy="0 0 0" />
+        <mass
+          value="303.81" />
+        <inertia
+          ixx="24.45402173"
+          ixy="-0.58037596"
+          ixz="-2.46563321"
+          iyy="20.71802091"
+          iyz="2.40454026"
+          izz="9.01610712" />
+      </inertial>
+      <visual>
+        <origin
+          xyz="0 0 0"
+          rpy="0 0 0" />
+        <geometry>
+          <mesh
+            filename="package://nj_220_2_7_gazebo/meshes/link_3.STL" />
+        </geometry>
+        <material
+          name="">
+          <color
+            rgba="1 0 0 1" />
+        </material>
+      </visual>
+      <collision>
+        <origin
+          xyz="0 0 0"
+          rpy="0 0 0" />
+        <geometry>
+          <mesh
+            filename="package://nj_220_2_7_gazebo/meshes/link_3.STL" />
+        </geometry>
+      </collision>
+    </link>
+    <joint name="${prefix}joint_3m" type="revolute">
+      <origin
+        xyz="0 0 0"
+        rpy="0 0 0" />
+      <parent
+        link="${prefix}link_3_virtual" />
+      <child
+        link="${prefix}link_3" />
+      <axis
+        xyz="0 1 0" />
+      <limit
+        lower="-6.2831853"
+        upper="6.2831853"
+        effort="0"
+        velocity="0" />
+      <mimic joint="${prefix}joint_3" multiplier="-1" offset="0" />
+    </joint>
+  </xacro:if>
+  <xacro:if value="${type == 'sdf'}">
+    <link name="${prefix}link_3">
+      <inertial>
+        <origin
+          xyz="-0.04239 0.01939 0.2104"
+          rpy="0 0 0" />
+        <mass
+          value="303.81" />
+        <inertia
+          ixx="24.45402173"
+          ixy="-0.58037596"
+          ixz="-2.46563321"
+          iyy="20.71802091"
+          iyz="2.40454026"
+          izz="9.01610712" />
+      </inertial>
+      <visual>
+        <origin
+          xyz="0 0 0"
+          rpy="0 0 0" />
+        <geometry>
+          <mesh
+            filename="package://nj_220_2_7_gazebo/meshes/link_3.STL" />
+        </geometry>
+        <material
+          name="">
+          <color
+            rgba="1 0 0 1" />
+        </material>
+      </visual>
+      <collision>
+        <origin
+          xyz="0 0 0"
+          rpy="0 0 0" />
+        <geometry>
+          <mesh
+            filename="package://nj_220_2_7_gazebo/meshes/link_3.STL" />
+        </geometry>
+      </collision>
+    </link>
+    <joint name="${prefix}joint_l2_l3" type="revolute">
+       <origin xyz="0 0 1.175" rpy="0 0 0" />
+       <parent link="${prefix}link_2" />
+       <child link="${prefix}link_3" />
+       <axis xyz="0 1 0" />
+       <limit
+         lower="-6.2831853"
+         upper="6.2831853"
+         effort="100000"
+         velocity="${joint_6_vel_limit}" />
+    </joint>
+  </xacro:if>
   <link name="${prefix}link_4">
     <inertial>
@@ -384,32 +464,18 @@
       velocity="${joint_6_vel_limit}" />
   </joint>
-  <link name="${prefix}link_3_virtual">
-   </link>
-  <joint name="${prefix}joint_2m" type="revolute">
-     <origin xyz="0 0 1.175" rpy="0 0 0" />
-     <parent link="${prefix}link_2" />
-     <child link="${prefix}link_3_virtual" />
-     <axis xyz="0 1 0" />
-     <mimic joint="${prefix}joint_2" multiplier="-1" offset="0" />
-     <limit
-       lower="-6.2831853"
-       upper="6.2831853"
-       effort="100000"
-       velocity="${joint_6_vel_limit}" />
-  </joint>
   <link name="${prefix}link_2_1">
      <inertial>
        <origin
-         xyz="0.14943 -0.0063786 0.023924"
+         xyz="-0.14831 0.02392 -0.01938"
          rpy="0 0 0" />
        <mass
          value="41.905" />
        <inertia
-         ixx="0.18520588"
-         ixy="-0.07064049"
-         ixz="0.17218606"
-         iyy="1.70899486"
-         iyz="-0.00657138"
-         izz="1.77577899" />
+         ixx="0.20904736"
+         ixy="-0.17095810"
+         ixz="0.20186889"
+         iyy="1.77577938"
+         iyz="-0.02155338"
+         izz="1.68515339" />
      </inertial>
      <visual>
@@ -437,70 +503,173 @@
      </collision>
    </link>
-  <joint name="${prefix}joint_2_1" type="revolute">
-     <origin xyz="0.400 -0.1945 0.499" rpy="1.570796327 0.087266 3.141592654" />
+  <joint name="${prefix}joint_3" type="revolute">
+     <origin xyz="0.400 -0.1945 0.499" rpy="0 0 0" />
      <parent link="${prefix}link_1" />
      <child link="${prefix}link_2_1" />
-     <axis xyz="0 0 1" />
+     <axis xyz="0 -1 0" />
      <limit
-       lower="-6.2831853"
-       upper="6.2831853"
-       effort="0"
-       velocity="0" />
-       <mimic joint="${prefix}joint_3" multiplier="-1" offset="0" />
+       lower="-4.468042885"
+       upper="0.174532925"
+       effort="${joint_3_eff_limit}"
+       velocity="${joint_3_vel_limit}" />
    </joint>
-  <link name="${prefix}link_2_2_virtual"></link>
-  <joint name="${prefix}joint_2_2" type="continuous">
-    <origin
-      xyz="0.350 0 0.015"
-      rpy="0 0 0.087266" />
-    <parent
-      link="${prefix}link_2_1" />
-    <child
-      link="${prefix}link_2_2_virtual" />
-    <axis
-      xyz="0 0 1" />
-    <mimic joint="${prefix}joint_3" multiplier="1" offset="0"/>
-  </joint>
-  <link name="${prefix}link_2_2">
-    <inertial>
-      <origin
-        xyz="0.06443 0.51885 0.01485"
-        rpy="0 0 0" />
-      <mass
-        value="60.72" />
-      <inertia
-        ixx="21.93937071"
-        ixy="1.89190480"
-        ixz="0.05733724"
-        iyy="0.41028863"
-        iyz="0.47064670"
-        izz="22.27041146" />
-    </inertial>
-    <visual>
-      <origin
-        xyz="0 0 0"
-        rpy="0 0 0" />
-      <geometry>
-        <mesh
-          filename="package://nj_220_2_7_gazebo/meshes/link_2_2.STL" />
-      </geometry>
-    </visual>
-    <collision>
-      <origin
-        xyz="0 0 0"
-        rpy="0 0 0" />
-      <geometry>
-        <mesh
-          filename="package://nj_220_2_7_gazebo/meshes/link_2_2.STL" />
-      </geometry>
-    </collision>
-  </link>
-  <joint name="${prefix}joint_2_3" type="continuous">
-    <origin xyz="0.0 0.0 0.0" rpy="0 0 0" />
-    <parent link="${prefix}link_2_2_virtual" />
-    <child link="${prefix}link_2_2" />
-    <axis xyz="0 0 1" />
-    <mimic joint="${prefix}joint_2" multiplier="1" offset="0"/>
-  </joint>
+  <xacro:if value="${type == 'urdf'}">
+    <link name="${prefix}link_2_2_virtual">
+      <inertial>
+        <origin xyz="0 0 0" rpy="0 0 0" />
+        <mass value="0.01" />
+        <inertia
+          ixx="0.00001"
+          ixy="0.00000"
+          ixz="0.00000"
+          iyy="0.00001"
+          iyz="0.00000"
+          izz="0.00000" />
+      </inertial>
+    </link>
+    <joint name="${prefix}joint_2_1" type="continuous">
+      <origin
+        xyz="-0.34867 0.015 -0.0305"
+        rpy="0 0 0" />
+      <parent link="${prefix}link_2_1" />
+      <child link="${prefix}link_2_2_virtual" />
+      <axis xyz="0 1 0" />
+      <mimic joint="${prefix}joint_3" multiplier="1" offset="0"/>
+    </joint>
+    <link name="${prefix}link_2_2">
+      <inertial>
+        <origin
+          xyz="-0.06443 0.01485 0.51885"
+          rpy="0 0 0" />
+        <mass
+          value="60.72" />
+        <inertia
+          ixx="21.93937071"
+          ixy="-0.05733724"
+          ixz="-1.89190480"
+          iyy="22.27041146"
+          iyz="0.47064670"
+          izz="0.41028863" />
+      </inertial>
+      <visual>
+        <origin
+          xyz="0 0 0"
+          rpy="0 0 0" />
+        <geometry>
+          <mesh
+            filename="package://nj_220_2_7_gazebo/meshes/link_2_2.STL" />
+        </geometry>
+      </visual>
+      <collision>
+        <origin
+          xyz="0 0 0"
+          rpy="0 0 0" />
+        <geometry>
+          <mesh
+            filename="package://nj_220_2_7_gazebo/meshes/link_2_2.STL" />
+        </geometry>
+      </collision>
+    </link>
+    <joint name="${prefix}joint_2_2" type="continuous">
+      <origin xyz="0.0 0.0 0.0" rpy="0 0 0" />
+      <parent link="${prefix}link_2_2_virtual" />
+      <child link="${prefix}link_2_2" />
+      <axis xyz="0 1 0" />
+      <mimic joint="${prefix}joint_2" multiplier="1" offset="0"/>
+    </joint>
+  </xacro:if>
+  <xacro:if value="${type == 'sdf'}">
+    <link name="${prefix}link_2_2">
+      <inertial>
+        <origin
+          xyz="-0.06443 0.01485 0.51885"
+          rpy="0 0 0" />
+        <mass
+          value="60.72" />
+        <inertia
+          ixx="21.93937071"
+          ixy="-0.05733724"
+          ixz="-1.89190480"
+          iyy="22.27041146"
+          iyz="0.47064670"
+          izz="0.41028863" />
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