Commit message: pybullet version, ready to tests

File: nj_220_2_7_description/urdf/nj_220_2_7.xacro (robot description, xacro)
@@ -1,6 +1,6 @@
 <?xml version="1.0" ?>
-<robot xmlns:xacro="http://ros.org/wiki/xacro">
-<!-- <xacro:macro name="nj_220_2_7" params="prefix:='' interface:=hardware_interface/EffortJointInterface type:=urdf"> -->
-  <xacro:macro name="nj_220_2_7" params="prefix:='' interface:=hardware_interface/PositionJointInterface type:=urdf">
+<robot name="nj_220_2_7" xmlns:xacro="http://ros.org/wiki/xacro">
+<xacro:macro name="nj_220_2_7" params="prefix:='' interface:=hardware_interface/EffortJointInterface type:=rviz">
+<!-- <xacro:macro name="nj_220_2_7" params="prefix:='' interface:=hardware_interface/PositionJointInterface type:=urdf"> -->
   <xacro:property name="joint_1_vel_limit" value="1.74533" />    <!--  100°/s -->
   <xacro:property name="joint_2_vel_limit" value="1.5708"  />    <!--  90°/s -->
@@ -164,32 +164,31 @@
       velocity="${joint_2_vel_limit}" />
   </joint>
-  <xacro:if value="${type == 'urdf'}">
-    <link name="${prefix}link_3_virtual">
-      <inertial>
-        <origin xyz="0 0 0" rpy="0 0 0" />
-        <mass value="0.01" />
-        <inertia
-          ixx="0.00001"
-          ixy="0.00000"
-          ixz="0.00000"
-          iyy="0.00001"
-          iyz="0.00000"
-          izz="0.00000" />
-      </inertial>
-    </link>
-    <joint name="${prefix}joint_2m" type="revolute">
-       <origin xyz="0 0 1.175" rpy="0 0 0" />
-       <parent link="${prefix}link_2" />
-       <child link="${prefix}link_3_virtual" />
-       <axis xyz="0 1 0" />
-       <mimic joint="${prefix}joint_2" multiplier="-1" offset="0" />
-       <limit
-         lower="-6.2831853"
-         upper="6.2831853"
-         effort="100000"
-         velocity="${joint_6_vel_limit}" />
-    </joint>
-    <link name="${prefix}link_3">
-      <inertial>
+  <link name="${prefix}link_3_virtual">
+    <inertial>
+      <origin xyz="0 0 0" rpy="0 0 0" />
+      <mass value="0.01" />
+      <inertia
+        ixx="0.00001"
+        ixy="0.00000"
+        ixz="0.00000"
+        iyy="0.00001"
+        iyz="0.00000"
+        izz="0.00000" />
+    </inertial>
+  </link>
+  <joint name="${prefix}joint_2m" type="revolute">
+    <origin xyz="0 0 1.175" rpy="0 0 0" />
+    <parent link="${prefix}link_2" />
+    <child link="${prefix}link_3_virtual" />
+    <axis xyz="0 1 0" />
+    <mimic joint="${prefix}joint_2" multiplier="-1" offset="0" />
+    <limit
+      lower="-6.2831853"
+      upper="6.2831853"
+      effort="100000"
+      velocity="${joint_6_vel_limit}" />
+  </joint>
+  <link name="${prefix}link_3">
+    <inertial>
         <origin
           xyz="-0.04239 0.01939 0.2104"
@@ -205,5 +204,5 @@
           izz="9.01610712" />
       </inertial>
-      <visual>
+    <visual>
         <origin
           xyz="0 0 0"
@@ -219,5 +218,5 @@
         </material>
       </visual>
-      <collision>
+    <collision>
         <origin
           xyz="0 0 0"
@@ -228,5 +227,6 @@
         </geometry>
       </collision>
-    </link>
+  </link>
+  <xacro:if value="${type == 'pybullet'}">
     <joint name="${prefix}joint_3m" type="revolute">
       <origin
@@ -247,54 +247,20 @@
     </joint>
   </xacro:if>
-  <xacro:if value="${type == 'sdf'}">
-    <link name="${prefix}link_3">
-      <inertial>
-        <origin
-          xyz="-0.04239 0.01939 0.2104"
-          rpy="0 0 0" />
-        <mass
-          value="303.81" />
-        <inertia
-          ixx="24.45402173"
-          ixy="-0.58037596"
-          ixz="-2.46563321"
-          iyy="20.71802091"
-          iyz="2.40454026"
-          izz="9.01610712" />
-      </inertial>
-      <visual>
-        <origin
-          xyz="0 0 0"
-          rpy="0 0 0" />
-        <geometry>
-          <mesh
-            filename="package://nj_220_2_7_gazebo/meshes/link_3.STL" />
-        </geometry>
-        <material
-          name="">
-          <color
-            rgba="1 0 0 1" />
-        </material>
-      </visual>
-      <collision>
-        <origin
-          xyz="0 0 0"
-          rpy="0 0 0" />
-        <geometry>
-          <mesh
-            filename="package://nj_220_2_7_gazebo/meshes/link_3.STL" />
-        </geometry>
-      </collision>
-    </link>
-    <joint name="${prefix}joint_l2_l3" type="revolute">
-       <origin xyz="0 0 1.175" rpy="0 0 0" />
-       <parent link="${prefix}link_2" />
-       <child link="${prefix}link_3" />
-       <axis xyz="0 1 0" />
-       <limit
-         lower="-6.2831853"
-         upper="6.2831853"
-         effort="100000"
-         velocity="${joint_6_vel_limit}" />
+  <xacro:if value="${type == 'rviz'}">
+    <joint name="${prefix}joint_3" type="revolute">
+      <origin
+        xyz="0 0 0"
+        rpy="0 0 0" />
+      <parent
+        link="${prefix}link_3_virtual" />
+      <child
+        link="${prefix}link_3" />
+      <axis
+        xyz="0 -1 0" />
+      <limit
+        lower="-4.468042885"
+        upper="0.174532925"
+        effort="${joint_3_eff_limit}"
+        velocity="${joint_3_vel_limit}" />
     </joint>
   </xacro:if>
@@ -465,212 +431,70 @@
   </joint>
   <link name="${prefix}link_2_1">
-     <inertial>
-       <origin
-         xyz="-0.14831 0.02392 -0.01938"
-         rpy="0 0 0" />
-       <mass
-         value="41.905" />
-       <inertia
-         ixx="0.20904736"
-         ixy="-0.17095810"
-         ixz="0.20186889"
-         iyy="1.77577938"
-         iyz="-0.02155338"
-         izz="1.68515339" />
-     </inertial>
-     <visual>
-       <origin
-         xyz="0 0 0"
-         rpy="0 0 0" />
-       <geometry>
-         <mesh
-           filename="package://nj_220_2_7_gazebo/meshes/link_2_1.STL" />
-       </geometry>
-       <material
-         name="">
-         <color
-           rgba="1 0 0 1" />
-       </material>
-     </visual>
-     <collision>
-       <origin
-         xyz="0 0 0"
-         rpy="0 0 0" />
-       <geometry>
-         <mesh
-           filename="package://nj_220_2_7_gazebo/meshes/link_2_1.STL" />
-       </geometry>
-     </collision>
-   </link>
-  <joint name="${prefix}joint_3" type="revolute">
-     <origin xyz="0.400 -0.1945 0.499" rpy="0 0 0" />
-     <parent link="${prefix}link_1" />
-     <child link="${prefix}link_2_1" />
-     <axis xyz="0 -1 0" />
-     <limit
+    <inertial>
+      <origin
+        xyz="-0.14831 0.02392 -0.01938"
+        rpy="0 0 0" />
+      <mass
+        value="41.905" />
+      <inertia
+        ixx="0.20904736"
+        ixy="-0.17095810"
+        ixz="0.20186889"
+        iyy="1.77577938"
+        iyz="-0.02155338"
+        izz="1.68515339" />
+    </inertial>
+    <visual>
+      <origin
+        xyz="0 0 0"
+        rpy="0 0 0" />
+      <geometry>
+        <mesh
+          filename="package://nj_220_2_7_gazebo/meshes/link_2_1.STL" />
+      </geometry>
+      <material
+        name="">
+        <color
+          rgba="1 0 0 1" />
+      </material>
+    </visual>
+    <collision>
+      <origin
+        xyz="0 0 0"
+        rpy="0 0 0" />
+      <geometry>
+        <mesh
+          filename="package://nj_220_2_7_gazebo/meshes/link_2_1.STL" />
+      </geometry>
+    </collision>
+  </link>
+  <xacro:if value="${type == 'pybullet'}">
+    <joint name="${prefix}joint_3" type="revolute">
+      <origin xyz="0.400 -0.1945 0.499" rpy="0 0 0" />
+      <parent link="${prefix}link_1" />
+      <child link="${prefix}link_2_1" />
+      <axis xyz="0 -1 0" />
+      <limit
        lower="-4.468042885"
        upper="0.174532925"
        effort="${joint_3_eff_limit}"
        velocity="${joint_3_vel_limit}" />
-   </joint>
-  <xacro:if value="${type == 'urdf'}">
-    <link name="${prefix}link_2_2_virtual">
-      <inertial>
-        <origin xyz="0 0 0" rpy="0 0 0" />
-        <mass value="0.01" />
-        <inertia
-          ixx="0.00001"
-          ixy="0.00000"
-          ixz="0.00000"
-          iyy="0.00001"
-          iyz="0.00000"
-          izz="0.00000" />
-      </inertial>
-    </link>
-    <joint name="${prefix}joint_2_1" type="continuous">
-      <origin
-        xyz="-0.34867 0.015 -0.0305"
-        rpy="0 0 0" />
-      <parent link="${prefix}link_2_1" />
-      <child link="${prefix}link_2_2_virtual" />
-      <axis xyz="0 1 0" />
-      <mimic joint="${prefix}joint_3" multiplier="1" offset="0"/>
-    </joint>
-    <link name="${prefix}link_2_2">
-      <inertial>
-        <origin
-          xyz="-0.06443 0.01485 0.51885"
-          rpy="0 0 0" />
-        <mass
-          value="60.72" />
-        <inertia
-          ixx="21.93937071"
-          ixy="-0.05733724"
-          ixz="-1.89190480"
-          iyy="22.27041146"
-          iyz="0.47064670"
-          izz="0.41028863" />
-      </inertial>
-      <visual>
-        <origin
-          xyz="0 0 0"
-          rpy="0 0 0" />
-        <geometry>
-          <mesh
-            filename="package://nj_220_2_7_gazebo/meshes/link_2_2.STL" />
-        </geometry>
-      </visual>
-      <collision>
-        <origin
-          xyz="0 0 0"
-          rpy="0 0 0" />
-        <geometry>
-          <mesh
-            filename="package://nj_220_2_7_gazebo/meshes/link_2_2.STL" />
-        </geometry>
-      </collision>
-    </link>
-    <joint name="${prefix}joint_2_2" type="continuous">
-      <origin xyz="0.0 0.0 0.0" rpy="0 0 0" />
-      <parent link="${prefix}link_2_2_virtual" />
-      <child link="${prefix}link_2_2" />
-      <axis xyz="0 1 0" />
-      <mimic joint="${prefix}joint_2" multiplier="1" offset="0"/>
     </joint>
   </xacro:if>
-  <xacro:if value="${type == 'sdf'}">
-    <link name="${prefix}link_2_2">
-      <inertial>
-        <origin
-          xyz="-0.06443 0.01485 0.51885"
-          rpy="0 0 0" />
-        <mass
-          value="60.72" />
-        <inertia
-          ixx="21.93937071"
-          ixy="-0.05733724"
-          ixz="-1.89190480"
-          iyy="22.27041146"
-          iyz="0.47064670"
-          izz="0.41028863" />
-      </inertial>
-      <visual>
-        <origin
-          xyz="0 0 0"
-          rpy="0 0 0" />
-        <geometry>
-          <mesh
-            filename="package://nj_220_2_7_gazebo/meshes/link_2_2.STL" />
-        </geometry>
-      </visual>
-      <collision>
-        <origin
-          xyz="0 0 0"
-          rpy="0 0 0" />
-        <geometry>
-          <mesh
-            filename="package://nj_220_2_7_gazebo/meshes/link_2_2.STL" />
-        </geometry>
-      </collision>
-    </link>
-    <joint name="${prefix}joint_2_1" type="revolute">
-      <origin xyz="-0.34867 0.015 -0.0305" rpy="0 0 0" />
-      <parent link="${prefix}link_2_1" />
-      <child link="${prefix}link_2_2" />
-      <axis xyz="0 1 0" />
+  <xacro:if value="${type == 'rviz'}">
+    <joint name="${prefix}joint_3m" type="revolute">
+      <origin xyz="0.400 -0.1945 0.499" rpy="0 0 0" />
+      <parent link="${prefix}link_1" />
+      <child link="${prefix}link_2_1" />
+      <axis xyz="0 -1 0" />
       <limit
         lower="-6.2831853"
         upper="6.2831853"
-        effort="100000"
-        velocity="${joint_6_vel_limit}" />
+        effort="0"
+        velocity="0" />
+        <mimic joint="${prefix}joint_3" multiplier="1" offset="0" />
     </joint>
-    <link name="${prefix}link_2_3">
-      <inertial>
-        <origin xyz="0 0 0" rpy="0 0 0" />
-        <mass value="0.01" />
-        <inertia
-          ixx="0.00001"
-          ixy="0.00000"
-          ixz="0.00000"
-          iyy="0.00001"
-          iyz="0.00000"
-          izz="0.00000" />
-      </inertial>
-      <!-- <visual>
-        <origin xyz="0 0 0" rpy="0 0 0" />
-        <geometry>
-          <box size="0.1 0.1 0.1" />
-        </geometry>
-        <material name="Cyan">
-          <color rgba="0 1.0 1.0 1.0"/>
-        </material>
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