Commit message: to fix

File: nj_220_2_7_description/urdf/nj_220_2_7.xacro (robot description, xacro)
@@ -2,5 +2,4 @@
 <robot name="nj_220_2_7" xmlns:xacro="http://ros.org/wiki/xacro">
 <xacro:macro name="nj_220_2_7" params="prefix:='' interface:=hardware_interface/EffortJointInterface type:=rviz">
-<!-- <xacro:macro name="nj_220_2_7" params="prefix:='' interface:=hardware_interface/PositionJointInterface type:=urdf"> -->
   <xacro:property name="joint_1_vel_limit" value="1.74533" />    <!--  100°/s -->
   <xacro:property name="joint_2_vel_limit" value="1.5708"  />    <!--  90°/s -->
@@ -36,5 +35,5 @@
       <geometry>
         <mesh
-          filename="package://nj_220_2_7_gazebo/meshes/base_link.STL" />
+          filename="package://nj_220_2_7_description/meshes/base_link.STL" />
       </geometry>
       <material
@@ -50,5 +49,5 @@
       <geometry>
         <mesh
-          filename="package://nj_220_2_7_gazebo/meshes/base_link.STL" />
+          filename="package://nj_220_2_7_description/meshes/base_link.STL" />
       </geometry>
     </collision>
@@ -75,5 +74,5 @@
       <geometry>
         <mesh
-          filename="package://nj_220_2_7_gazebo/meshes/link_1.STL" />
+          filename="package://nj_220_2_7_description/meshes/link_1.STL" />
       </geometry>
       <material
@@ -89,5 +88,5 @@
       <geometry>
         <mesh
-          filename="package://nj_220_2_7_gazebo/meshes/link_1.STL" />
+          filename="package://nj_220_2_7_description/meshes/link_1.STL" />
       </geometry>
     </collision>
@@ -130,5 +129,5 @@
       <geometry>
         <mesh
-          filename="package://nj_220_2_7_gazebo/meshes/link_2.STL" />
+          filename="package://nj_220_2_7_description/meshes/link_2.STL" />
       </geometry>
       <material
@@ -144,5 +143,5 @@
       <geometry>
         <mesh
-          filename="package://nj_220_2_7_gazebo/meshes/link_2.STL" />
+          filename="package://nj_220_2_7_description/meshes/link_2.STL" />
       </geometry>
     </collision>
@@ -163,29 +162,4 @@
       effort="${joint_2_eff_limit}"
       velocity="${joint_2_vel_limit}" />
-  </joint>
-  <link name="${prefix}link_3_virtual">
-    <inertial>
-      <origin xyz="0 0 0" rpy="0 0 0" />
-      <mass value="0.01" />
-      <inertia
-        ixx="0.00001"
-        ixy="0.00000"
-        ixz="0.00000"
-        iyy="0.00001"
-        iyz="0.00000"
-        izz="0.00000" />
-    </inertial>
-  </link>
-  <joint name="${prefix}joint_2m" type="revolute">
-    <origin xyz="0 0 1.175" rpy="0 0 0" />
-    <parent link="${prefix}link_2" />
-    <child link="${prefix}link_3_virtual" />
-    <axis xyz="0 1 0" />
-    <mimic joint="${prefix}joint_2" multiplier="-1" offset="0" />
-    <limit
-      lower="-6.2831853"
-      upper="6.2831853"
-      effort="100000"
-      velocity="${joint_6_vel_limit}" />
   </joint>
   <link name="${prefix}link_3">
@@ -210,5 +184,5 @@
         <geometry>
           <mesh
-            filename="package://nj_220_2_7_gazebo/meshes/link_3.STL" />
+            filename="package://nj_220_2_7_description/meshes/link_3.STL" />
         </geometry>
         <material
@@ -224,15 +198,15 @@
         <geometry>
           <mesh
-            filename="package://nj_220_2_7_gazebo/meshes/link_3.STL" />
+            filename="package://nj_220_2_7_description/meshes/link_3.STL" />
         </geometry>
       </collision>
   </link>
   <xacro:if value="${type == 'pybullet'}">
-    <joint name="${prefix}joint_3m" type="revolute">
-      <origin
-        xyz="0 0 0"
+    <joint name="${prefix}free_joint" type="revolute">
+      <origin
+        xyz="0 0 1.175"
         rpy="0 0 0" />
       <parent
-        link="${prefix}link_3_virtual" />
+        link="${prefix}link_2" />
       <child
         link="${prefix}link_3" />
@@ -244,8 +218,32 @@
         effort="0"
         velocity="0" />
-      <mimic joint="${prefix}joint_3" multiplier="-1" offset="0" />
     </joint>
   </xacro:if>
   <xacro:if value="${type == 'rviz'}">
+    <link name="${prefix}link_3_virtual">
+      <inertial>
+        <origin xyz="0 0 0" rpy="0 0 0" />
+        <mass value="0.01" />
+        <inertia
+          ixx="0.00001"
+          ixy="0.00000"
+          ixz="0.00000"
+          iyy="0.00001"
+          iyz="0.00000"
+          izz="0.00000" />
+      </inertial>
+    </link>
+    <joint name="${prefix}joint_2m" type="revolute">
+      <origin xyz="0 0 1.175" rpy="0 0 0" />
+      <parent link="${prefix}link_2" />
+      <child link="${prefix}link_3_virtual" />
+      <axis xyz="0 1 0" />
+      <mimic joint="${prefix}joint_2" multiplier="-1" offset="0" />
+      <limit
+        lower="-6.2831853"
+        upper="6.2831853"
+        effort="100000"
+        velocity="${joint_6_vel_limit}" />
+    </joint>
     <joint name="${prefix}joint_3" type="revolute">
       <origin
@@ -286,5 +284,5 @@
       <geometry>
         <mesh
-          filename="package://nj_220_2_7_gazebo/meshes/link_4.STL" />
+          filename="package://nj_220_2_7_description/meshes/link_4.STL" />
       </geometry>
       <material
@@ -300,5 +298,5 @@
       <geometry>
         <mesh
-          filename="package://nj_220_2_7_gazebo/meshes/link_4.STL" />
+          filename="package://nj_220_2_7_description/meshes/link_4.STL" />
       </geometry>
     </collision>
@@ -341,5 +339,5 @@
       <geometry>
         <mesh
-          filename="package://nj_220_2_7_gazebo/meshes/link_5.STL" />
+          filename="package://nj_220_2_7_description/meshes/link_5.STL" />
       </geometry>
       <material
@@ -355,5 +353,5 @@
       <geometry>
         <mesh
-          filename="package://nj_220_2_7_gazebo/meshes/link_5.STL" />
+          filename="package://nj_220_2_7_description/meshes/link_5.STL" />
       </geometry>
     </collision>
@@ -396,5 +394,5 @@
       <geometry>
         <mesh
-          filename="package://nj_220_2_7_gazebo/meshes/link_6.STL" />
+          filename="package://nj_220_2_7_description/meshes/link_6.STL" />
       </geometry>
       <material
@@ -410,5 +408,5 @@
       <geometry>
         <mesh
-          filename="package://nj_220_2_7_gazebo/meshes/link_6.STL" />
+          filename="package://nj_220_2_7_description/meshes/link_6.STL" />
       </geometry>
     </collision>
@@ -451,5 +449,5 @@
       <geometry>
         <mesh
-          filename="package://nj_220_2_7_gazebo/meshes/link_2_1.STL" />
+          filename="package://nj_220_2_7_description/meshes/link_2_1.STL" />
       </geometry>
       <material
@@ -465,5 +463,50 @@
       <geometry>
         <mesh
-          filename="package://nj_220_2_7_gazebo/meshes/link_2_1.STL" />
+          filename="package://nj_220_2_7_description/meshes/link_2_1.STL" />
+      </geometry>
+    </collision>
+  </link>
+  <link name="${prefix}link_2_2">
+    <!-- <inertial>
+      <origin
+        xyz="-0.06443 0.01485 0.51885"
+        rpy="0 0 0" />
+      <mass
+        value="60.72" />
+      <inertia
+        ixx="21.93937071"
+        ixy="-0.05733724"
+        ixz="-1.89190480"
+        iyy="22.27041146"
+        iyz="0.47064670"
+        izz="0.41028863" />
+    </inertial> -->
+    <inertial>
+      <origin xyz="0 0 0" rpy="0 0 0" />
+      <mass value="0.01" />
+      <inertia
+        ixx="0.00001"
+        ixy="0.00000"
+        ixz="0.00000"
+        iyy="0.00001"
+        iyz="0.00000"
+        izz="0.00000" />
+    </inertial>
+    <visual>
+      <origin
+        xyz="0 0 0"
+        rpy="0 0 0" />
+      <geometry>
+        <mesh
+          filename="package://nj_220_2_7_description/meshes/link_2_2.STL" />
+      </geometry>
+    </visual>
+    <collision>
+      <origin
+        xyz="0 0 0"
+        rpy="0 0 0" />
+      <geometry>
+        <mesh
+          filename="package://nj_220_2_7_description/meshes/link_2_2.STL" />
       </geometry>
     </collision>
@@ -480,4 +523,15 @@
        effort="${joint_3_eff_limit}"
        velocity="${joint_3_vel_limit}" />
+    </joint>
+    <joint name="${prefix}joint_2_1" type="revolute">
+      <origin xyz="-0.34867 0.015 -0.0305" rpy="0 0 0" />
+      <parent link="${prefix}link_2_1" />
+      <child link="${prefix}link_2_2" />
+      <axis xyz="0 1 0" />
+      <limit
+        lower="-6.2831853"
+        upper="6.2831853"
+        effort="0"
+        velocity="0" />
     </joint>
   </xacro:if>
@@ -495,6 +549,42 @@
         <mimic joint="${prefix}joint_3" multiplier="1" offset="0" />
     </joint>
+    <link name="${prefix}link_2_2_virtual">
+      <inertial>
+        <origin xyz="0 0 0" rpy="0 0 0" />
+        <mass value="0.01" />
+        <inertia
+          ixx="0.00001"
+          ixy="0.00000"
+          ixz="0.00000"
+          iyy="0.00001"
+          iyz="0.00000"
+          izz="0.00000" />
+      </inertial>
+      <collision>
+        <origin xyz="0 ${0.05} 0" rpy="0 0 0" />
+        <geometry>
+          <box size="0.01 0.1 0.01"/>
+        </geometry>
+        <material name="aluminium">
+          <color rgba="${132/256} ${135/256} ${137/256} 1" />
+        </material>
+      </collision>
+    </link>
+    <joint name="${prefix}joint_2_1" type="continuous">
+      <origin xyz="-0.34867 0.015 -0.0305" rpy="0 0 0" />
+      <parent link="${prefix}link_2_1" />
+      <child link="${prefix}link_2_2_virtual" />
+      <axis xyz="0 1 0" />
+      <mimic joint="${prefix}joint_3" multiplier="1" offset="0"/>
+    </joint>
+    <joint name="${prefix}joint_2_2" type="continuous">
+      <origin xyz="0.0 0.0 0.0" rpy="0 0 0" />
+      <parent link="${prefix}link_2_2_virtual" />
+      <child link="${prefix}link_2_2" />
+      <axis xyz="0 1 0" />
+      <mimic joint="${prefix}joint_2" multiplier="1" offset="0"/>
+    </joint>
   </xacro:if>
-  <link name="${prefix}link_2_2_virtual">
+  <link name="${prefix}link_2_3">
     <inertial>
       <origin xyz="0 0 0" rpy="0 0 0" />
@@ -508,54 +598,13 @@
         izz="0.00000" />
     </inertial>
-  </link>
-  <joint name="${prefix}joint_2_1" type="continuous">
-    <origin xyz="-0.34867 0.015 -0.0305" rpy="0 0 0" />
-    <parent link="${prefix}link_2_1" />
-    <child link="${prefix}link_2_2_virtual" />
-    <axis xyz="0 1 0" />
-    <mimic joint="${prefix}joint_3" multiplier="1" offset="0"/>
-  </joint>
-  <link name="${prefix}link_2_2">
-    <inertial>
-      <origin
-        xyz="-0.06443 0.01485 0.51885"
-        rpy="0 0 0" />
-      <mass
-        value="60.72" />
-      <inertia
-        ixx="21.93937071"
-        ixy="-0.05733724"
-        ixz="-1.89190480"
-        iyy="22.27041146"
-        iyz="0.47064670"
-        izz="0.41028863" />
-    </inertial>
-    <visual>
-      <origin
-        xyz="0 0 0"
-        rpy="0 0 0" />
-      <geometry>
-        <mesh
-          filename="package://nj_220_2_7_gazebo/meshes/link_2_2.STL" />
-      </geometry>
-    </visual>
-    <collision>
-      <origin
-        xyz="0 0 0"
-        rpy="0 0 0" />
-      <geometry>
-        <mesh
-          filename="package://nj_220_2_7_gazebo/meshes/link_2_2.STL" />
-      </geometry>
-    </collision>
-  </link>
-  <joint name="${prefix}joint_2_2" type="continuous">
-    <origin xyz="0.0 0.0 0.0" rpy="0 0 0" />
-    <parent link="${prefix}link_2_2_virtual" />
-    <child link="${prefix}link_2_2" />
-    <axis xyz="0 1 0" />
-    <mimic joint="${prefix}joint_2" multiplier="1" offset="0"/>
-  </joint>
-  <link name="${prefix}link_2_3">
+    <collision>
+      <origin xyz="0 0 0" rpy="0 0 0" />
+      <geometry>
+        <box size="0.01 0.5 0.01"/>
+      </geometry>
+      <material name="aluminium">
+        <color rgba="${132/256} ${135/256} ${137/256} 1" />
+      </material>
+    </collision>
     </link>
   <joint name="${prefix}joint_2_3" type="continuous">
@@ -564,14 +613,11 @@
     <child link="${prefix}link_2_3" />
     <axis xyz="0 1 0" />
+    <limit
+      lower="-6.2831853"
+      upper="6.2831853"
+      effort="0"
+      velocity="0" />
   </joint>
   <link name="${prefix}link_2_4">
-    </link>
-  <joint name="${prefix}joint_2_4" type="continuous">
-    <origin xyz="-0.34867 -0.1795 -0.0305" rpy="0 0 0" />
-    <parent link="${prefix}link_3" />
-    <child link="${prefix}link_2_4" />
-    <axis xyz="0 1 0" />
-  </joint>
-  <link name="${prefix}flange">
     <inertial>
       <origin xyz="0 0 0" rpy="0 0 0" />
@@ -585,4 +631,33 @@
         izz="0.00000" />
     </inertial>
+    <collision>
+      <origin xyz="0 0 0" rpy="0 0 0" />
+      <geometry>
+        <box size="0.01 0.5 0.01"/>
+      </geometry>
+      <material name="aluminium">
+        <color rgba="${132/256} ${135/256} ${137/256} 1" />
+      </material>
+    </collision>
+    </link>
+  <joint name="${prefix}joint_2_4" type="fixed">
+    <origin xyz="-0.34867 -0.1795 -0.0305" rpy="0 0 0" />
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
File: nj_220_2_7_description/urdf/nj_220_2_7_pybullet.urdf (robot description, URDF)
Before this commit: robot nj_220_2_7, 21 links, 20 joints
Links:
- removed link flange
- removed link link_2_2_virtual
- removed link link_3_virtual
- removed link link_4
- removed link link_5
- removed link link_6
- link base_link: geometry collision mesh filename=package://nj_220_2_7_description/meshes/base_link.STL; visual mesh filename=package://nj_220_2_7_description/meshes/base_link.STL
- link external_piece: geometry collision mesh filename=package://nj_220_2_7_description/meshes/external_part.STL; visual mesh filename=package://nj_220_2_7_description/meshes/external_part.STL
- link link_1: geometry collision mesh filename=package://nj_220_2_7_description/meshes/link_1.STL; visual mesh filename=package://nj_220_2_7_description/meshes/link_1.STL
- link link_2: geometry collision mesh filename=package://nj_220_2_7_description/meshes/link_2.STL; visual mesh filename=package://nj_220_2_7_description/meshes/link_2.STL
- link link_2_1: geometry collision mesh filename=package://nj_220_2_7_description/meshes/link_2_1.STL; visual mesh filename=package://nj_220_2_7_description/meshes/link_2_1.STL
- link link_2_2: mass 60.72 -> 0.01; geometry collision mesh filename=package://nj_220_2_7_description/meshes/link_2_2.STL; visual mesh filename=package://nj_220_2_7_description/meshes/link_2_2.STL
- link link_2_3: mass None -> 0.01; geometry collision box size=0.01 0.5 0.01
- link link_2_4: mass None -> 0.01; geometry collision box size=0.01 0.5 0.01
- link link_3: geometry collision mesh filename=package://nj_220_2_7_description/meshes/link_3.STL; visual mesh filename=package://nj_220_2_7_description/meshes/link_3.STL
- link motor_1: geometry collision mesh filename=package://nj_220_2_7_description/meshes/motor_80.STL; visual mesh filename=package://nj_220_2_7_description/meshes/motor_80.STL
- link motor_2: geometry collision mesh filename=package://nj_220_2_7_description/meshes/motor_90.STL; visual mesh filename=package://nj_220_2_7_description/meshes/motor_90.STL
- link motor_3: geometry collision mesh filename=package://nj_220_2_7_description/meshes/motor_80.STL; visual mesh filename=package://nj_220_2_7_description/meshes/motor_80.STL
- link motor_4: geometry collision mesh filename=package://nj_220_2_7_description/meshes/motor_50.STL; visual mesh filename=package://nj_220_2_7_description/meshes/motor_50.STL
- link motor_5: geometry collision mesh filename=package://nj_220_2_7_description/meshes/motor_50.STL; visual mesh filename=package://nj_220_2_7_description/meshes/motor_50.STL
- link motor_6: geometry collision mesh filename=package://nj_220_2_7_description/meshes/motor_50.STL; visual mesh filename=package://nj_220_2_7_description/meshes/motor_50.STL
Joints:
- removed joint joint_2_2
- removed joint joint_2m
- removed joint joint_3m
- removed joint joint_4
- removed joint joint_5
- removed joint joint_6
- removed joint link_6_to_flange
- added joint free_joint: type revolute, parent link_2, child link_3, origin xyz=0 0 1.175 rpy=0 0 0, axis 0 1 0, limit lower=-6.2831853 upper=6.2831853 effort=0 velocity=0
- joint joint_2_1: child link_2_2_virtual -> link_2_2; limit (none) -> lower=-6.2831853 upper=6.2831853 effort=0 velocity=0; mimic joint=joint_3 multiplier=1 offset=0 -> (none); type continuous -> revolute
- joint joint_2_3: limit (none) -> lower=-6.2831853 upper=6.2831853 effort=0 velocity=0
- joint joint_2_4: type continuous -> fixed

File: nj_220_2_7_description/urdf/nj_220_2_7_rviz.xacro (robot description, xacro)
@@ -1,9 +1,9 @@
 <?xml version="1.0"?>
 <robot name="nj_220_2_7" xmlns:xacro="http://www.ros.org/wiki/xacro">
-<xacro:include filename="$(find nj_220_2_7_description)/urdf/nj_220_2_7.xacro" />
-<xacro:property name="prefix" value="''" />
-<xacro:property name="type"   value="'rviz'" />
-<link name="world"/>
+  <xacro:include filename="$(find nj_220_2_7_description)/urdf/nj_220_2_7.xacro" />
+  <xacro:property name="prefix" value="''" />
+  <xacro:property name="type"   value="'rviz'" />
   <xacro:nj_220_2_7 prefix="${prefix}" type="${type}"/>
+  <link name="world"/>
   <joint name="${prefix}world_to_base_link" type="fixed">
       <origin
